Commit message: mesh updated

File: catarm_description/urdf/arm/CAT-ARM-001.urdf.xacro (robot description, xacro)
@@ -27,5 +27,5 @@
       <parent link="${prefix}arm/link0"/>
       <child link="${prefix}arm/link1"/>
-      <origin xyz="0 0 0.1" rpy="0 0 0"/>
+      <origin xyz="0 0 0.08" rpy="0 0 0"/>
       <axis xyz="0 0 1"/>
       <limit lower="${-90*M_PI/180}" upper="${90*M_PI/180}" effort="6"
@@ -48,5 +48,5 @@
       <parent link="${prefix}arm/link1"/>
       <child link="${prefix}arm/link2"/>
-      <origin xyz="0 0 0.1" rpy="0 ${-90*M_PI/180} ${180*M_PI/180}"/>
+      <origin xyz="0 0 0.08" rpy="${90*M_PI/180} 0 ${90*M_PI/180}"/>
       <axis xyz="0 0 1"/>
       <limit lower="${-90*M_PI/180}" upper="${90*M_PI/180}" effort="6"
@@ -69,5 +69,5 @@
       <parent link="${prefix}arm/link2"/>
       <child link="${prefix}arm/link3"/>
-      <origin xyz="0.5 0 0" rpy="0 0 0"/>
+      <origin xyz="0 0.4 0" rpy="0 0 0"/>
       <axis xyz="0 0 1"/>
       <limit lower="${-135*M_PI/180}" upper="${135*M_PI/180}" effort="6"
@@ -90,5 +90,5 @@
       <parent link="${prefix}arm/link3"/>
       <child link="${prefix}arm/link4"/>
-      <origin xyz="0.5 0 0" rpy="0 0 0"/>
+      <origin xyz="0 0.4 0" rpy="0 0 0"/>
       <axis xyz="0 0 1"/>
       <limit lower="${-90*M_PI/180}" upper="${90*M_PI/180}" effort="6"
@@ -111,5 +111,5 @@
       <parent link="${prefix}arm/link4"/>
       <child link="${prefix}arm/link5"/>
-      <origin xyz="0.18 0 0" rpy="0 ${90*M_PI/180} 0"/>
+      <origin xyz="0 0.04 0" rpy="${-90*M_PI/180} 0 0"/>
       <axis xyz="0 0 1"/>
       <limit lower="${-180*M_PI/180}" upper="${180*M_PI/180}" effort="6"
@@ -132,5 +132,5 @@
       <parent link="${prefix}arm/link5"/>
       <child link="${prefix}arm/link_tip"/>
-      <origin xyz="0.18 0 0" rpy="0 0 0"/>
+      <origin xyz="0 0 0.02" rpy="0 0 0"/>
     </joint>
     <link name="${prefix}arm/link_tip"/>

File: catarm_description/urdf/gripper/CAT-GRIPPER-001.urdf.xacro (robot description, xacro)
@@ -24,10 +24,10 @@
       </collision>
     </link>
-    <joint name="${prefix}gripper/joint1" type="revolute">
+    <joint name="${prefix}gripper/joint1" type="prismatic">
       <parent link="${prefix}gripper/base_link"/>
       <child link="${prefix}gripper/finger1"/>
-      <origin xyz="0.112 0 0" rpy="${90*M_PI/180} 0 ${90*M_PI/180}"/>
+      <origin xyz="0 0 0.01" rpy="${90*M_PI/180} 0 0"/>
       <axis xyz="0 0 1"/>
-      <limit lower="${-25*M_PI/180}" upper="${25*M_PI/180}" effort="6"
+      <limit lower="0" upper="0.05" effort="6"
               velocity="5" acceleration="5"/>
     </joint>
@@ -45,12 +45,12 @@
       </collision>
     </link>
-    <joint name="${prefix}gripper/joint2" type="revolute">
+    <joint name="${prefix}gripper/joint2" type="prismatic">
       <parent link="${prefix}gripper/base_link"/>
       <child link="${prefix}gripper/finger2"/>
-      <origin xyz="0.0956 0 0" rpy="${-90*M_PI/180} 0 ${-90*M_PI/180}"/>
+      <origin xyz="0 0 0.01" rpy="${90*M_PI/180} 0 0"/>
       <axis xyz="0 0 1"/>
-      <limit lower="${-150*M_PI/180}" upper="${150*M_PI/180}" effort="6"
+      <limit lower="0" upper="0.05" effort="6"
               velocity="5" acceleration="5"/>
-      <mimic joint="${prefix}gripper/joint1" multiplier="1" offset="0" />
+      <mimic joint="${prefix}gripper/joint1" multiplier="-1" offset="0" />
     </joint>
     <link name="${prefix}gripper/finger2">
@@ -70,5 +70,5 @@
       <parent link="${prefix}gripper/base_link"/>
       <child link="${prefix}gripper/link_tip"/>
-      <origin xyz="0.18 0 0" rpy="0 0 0"/>
+      <origin xyz="0 0 0.03" rpy="0 0 0"/>
     </joint>
     <link name="${prefix}gripper/link_tip"/>
