Commit message: fix shooting plan

File: catchrobo_description/urdf/arm.urdf.xacro (robot description, xacro)
@@ -30,5 +30,5 @@
       <origin xyz="0 0 0.1675" rpy="0 0 0"/>
       <axis xyz="0 0 1"/>
-      <limit lower="${-160*M_PI/180}" upper="${160*M_PI/180}" effort="6"
+      <limit lower="${-180*M_PI/180}" upper="${160*M_PI/180}" effort="6"
               velocity="5" acceleration="5"/>
     </joint>

Commit message: urdf

File: catchrobo_description/urdf/arm.urdf.xacro (robot description, xacro)
@@ -51,5 +51,5 @@
       <origin xyz="0 0 0" rpy="${90*M_PI/180} 0 0"/>
       <axis xyz="0 0 1"/>
-      <limit lower="${-90*M_PI/180}" upper="${90*M_PI/180}" effort="6"
+      <limit lower="${-90*M_PI/180}" upper="${59*M_PI/180}" effort="6"
               velocity="5" acceleration="5"/>
     </joint>

Commit message: gui

File: catchrobo_description/urdf/arm.urdf.xacro (robot description, xacro)
@@ -51,5 +51,5 @@
       <origin xyz="0 0 0" rpy="${90*M_PI/180} 0 0"/>
       <axis xyz="0 0 1"/>
-      <limit lower="${-90*M_PI/180}" upper="${59*M_PI/180}" effort="6"
+      <limit lower="${-90*M_PI/180}" upper="${60*M_PI/180}" effort="6"
               velocity="5" acceleration="5"/>
     </joint>

Commit message: vel change

File: catchrobo_description/urdf/arm.urdf.xacro (robot description, xacro)
@@ -51,5 +51,5 @@
       <origin xyz="0 0 0" rpy="${90*M_PI/180} 0 0"/>
       <axis xyz="0 0 1"/>
-      <limit lower="${-90*M_PI/180}" upper="${60*M_PI/180}" effort="6"
+      <limit lower="${-90*M_PI/180}" upper="${90*M_PI/180}" effort="6"
               velocity="5" acceleration="5"/>
     </joint>

Commit message: final version of 10/02

File: catchrobo_description/urdf/arm.urdf.xacro (robot description, xacro)
@@ -30,5 +30,5 @@
       <origin xyz="0 0 0.1675" rpy="0 0 0"/>
       <axis xyz="0 0 1"/>
-      <limit lower="${-180*M_PI/180}" upper="${160*M_PI/180}" effort="6"
+      <limit lower="${-150*M_PI/180}" upper="${150*M_PI/180}" effort="6"
               velocity="5" acceleration="5"/>
     </joint>

Commit message: move on melodic

File: catchrobo_description/urdf/arm.urdf.xacro (robot description, xacro)
@@ -30,5 +30,5 @@
       <origin xyz="0 0 0.1675" rpy="0 0 0"/>
       <axis xyz="0 0 1"/>
-      <limit lower="${-150*M_PI/180}" upper="${150*M_PI/180}" effort="6"
+      <limit lower="${-180*M_PI/180}" upper="${180*M_PI/180}" effort="6"
               velocity="5" acceleration="5"/>
     </joint>

Commit message: move with collision check

File: catchrobo_description/urdf/arm.urdf.xacro (robot description, xacro)
@@ -30,5 +30,5 @@
       <origin xyz="0 0 0.1675" rpy="0 0 0"/>
       <axis xyz="0 0 1"/>
-      <limit lower="${-180*M_PI/180}" upper="${180*M_PI/180}" effort="6"
+      <limit lower="${-180*M_PI/180}" upper="${179*M_PI/180}" effort="6"
               velocity="5" acceleration="5"/>
     </joint>
@@ -114,5 +114,5 @@
       <origin xyz="0 0.046 0" rpy="${-90*M_PI/180} 0 0"/>
       <axis xyz="0 0 1"/>
-      <limit lower="${-160*M_PI/180}" upper="${160*M_PI/180}" effort="6"
+      <limit lower="${-180*M_PI/180}" upper="${179*M_PI/180}" effort="6"
               velocity="5" acceleration="5"/>
     </joint>

Commit message: ugokuyo!

File: catchrobo_description/urdf/arm.urdf.xacro (robot description, xacro)
@@ -30,5 +30,5 @@
       <origin xyz="0 0 0.1675" rpy="0 0 0"/>
       <axis xyz="0 0 1"/>
-      <limit lower="${-180*M_PI/180}" upper="${179*M_PI/180}" effort="6"
+      <limit lower="${-175*M_PI/180}" upper="${175*M_PI/180}" effort="6"
               velocity="5" acceleration="5"/>
     </joint>
@@ -51,5 +51,5 @@
       <origin xyz="0 0 0" rpy="${90*M_PI/180} 0 0"/>
       <axis xyz="0 0 1"/>
-      <limit lower="${-90*M_PI/180}" upper="${90*M_PI/180}" effort="6"
+      <limit lower="${-90*M_PI/180}" upper="${60*M_PI/180}" effort="6"
               velocity="5" acceleration="5"/>
     </joint>
@@ -114,5 +114,5 @@
       <origin xyz="0 0.046 0" rpy="${-90*M_PI/180} 0 0"/>
       <axis xyz="0 0 1"/>
-      <limit lower="${-180*M_PI/180}" upper="${179*M_PI/180}" effort="6"
+      <limit lower="${-175*M_PI/180}" upper="${175*M_PI/180}" effort="6"
               velocity="5" acceleration="5"/>
     </joint>

Commit message: a

File: catchrobo_description/urdf/arm.urdf.xacro (robot description, xacro)
@@ -114,5 +114,5 @@
       <origin xyz="0 0.046 0" rpy="${-90*M_PI/180} 0 0"/>
       <axis xyz="0 0 1"/>
-      <limit lower="${-175*M_PI/180}" upper="${175*M_PI/180}" effort="6"
+      <limit lower="${-180*M_PI/180}" upper="${179*M_PI/180}" effort="6"
               velocity="5" acceleration="5"/>
     </joint>

Commit message: blue ok

File: catchrobo_description/urdf/arm.urdf.xacro (robot description, xacro)
@@ -114,5 +114,5 @@
       <origin xyz="0 0.046 0" rpy="${-90*M_PI/180} 0 0"/>
       <axis xyz="0 0 1"/>
-      <limit lower="${-180*M_PI/180}" upper="${179*M_PI/180}" effort="6"
+      <limit lower="${-175*M_PI/180}" upper="${175*M_PI/180}" effort="6"
               velocity="5" acceleration="5"/>
     </joint>
