Commit message: [Minor] ビスコ干渉回避用に高さを変更 (feature_shooter_fixed_urdf)

File: catchrobo_description/urdf/shooter.urdf.xacro (robot description, xacro)
@@ -46,5 +46,5 @@
       <parent link="${prefix}shooter_base/base_link"/>
       <child link="${prefix}shooter/guide"/>
-      <origin xyz="0.3083 0.42041555 0.07832442" rpy="${-90*M_PI/180} ${35*M_PI/180} ${90*M_PI/180}"/>
+      <origin xyz="0.3083 0.4215627 0.07996272" rpy="${-90*M_PI/180} ${35*M_PI/180} ${90*M_PI/180}"/>
       <axis xyz="0 0 1"/>
       <limit lower="${-175*M_PI/180}" upper="${175*M_PI/180}" effort="6"

Commit message: [Minor] ビスコ干渉回避用に高さ変更 (feature_shooter_fixed_urdf)

File: catchrobo_description/urdf/shooter.urdf.xacro (robot description, xacro)
@@ -30,5 +30,5 @@
       <parent link="${prefix}shooter/base_link"/>
       <child link="${prefix}shooter/guide"/>
-      <origin xyz="0.3083 0.42041555 0.07832442" rpy="${-90*M_PI/180} ${35*M_PI/180} ${90*M_PI/180}"/>
+      <origin xyz="0.3083 0.4215627 0.07996272" rpy="${-90*M_PI/180} ${35*M_PI/180} ${90*M_PI/180}"/>
       <axis xyz="0 0 1"/>
       <limit lower="${-175*M_PI/180}" upper="${175*M_PI/180}" effort="6"

Commit message: shooter with rope_jig

File: catchrobo_description/urdf/shooter.urdf.xacro (robot description, xacro)
@@ -111,4 +111,22 @@
       </collision>
     </link>
+    <joint name="${prefix}sorter/wire_guide" type="fixed">
+      <parent link="${prefix}shooter/base_link"/>
+      <child link="${prefix}shooter/wire_guide"/>
+      <origin xyz="0 0.37 0.17" rpy="${90*M_PI/180} 0 ${180*M_PI/180}"/>
+    </joint>
+    <link name="${prefix}shooter/wire_guide">
+      <visual>
+        <geometry>
+          <mesh filename="package://catchrobo_description/mesh/shooter/visual/wire_guide.stl" scale="${visual_mesh_scale}"/>
+        </geometry>
+        <material name="white"/>
+      </visual>
+      <collision>
+        <geometry>
+          <mesh filename="package://catchrobo_description/mesh/shooter/collision/wire_guide.stl" scale="${collision_mesh_scale}"/>
+        </geometry>
+      </collision>
+    </link>
   </xacro:macro>
 </robot>
