Commit message: scara ver

File: catchrobo_description/urdf/scara.urdf.xacro (robot description, xacro)
@@ -93,5 +93,5 @@
       <origin xyz="0 0 -0.0403" rpy="0 0 0"/>
       <axis xyz="0 0 1"/>
-      <limit lower="0" upper="-0.25" effort="6"
+      <limit lower="-0.25" upper="0" effort="6"
               velocity="5" acceleration="5"/>
     </joint>

Commit message: scara mesh and urdf update added hardstop feature to driver

File: catchrobo_description/urdf/scara.urdf.xacro (robot description, xacro)
@@ -28,5 +28,5 @@
       <parent link="${prefix}arm/link0"/>
       <child link="${prefix}arm/link1"/>
-      <origin xyz="0 0 0.3375" rpy="0 0 0"/>
+      <origin xyz="0 0 0.3875" rpy="0 0 0"/>
       <axis xyz="0 0 1"/>
       <limit lower="${-160*M_PI/180}" upper="${160*M_PI/180}" effort="6"
@@ -97,5 +97,5 @@
       <parent link="${prefix}arm/link3"/>
       <child link="${prefix}arm/link4"/>
-      <origin xyz="0 0 -0.03295" rpy="0 0 0"/>
+      <origin xyz="0 0 -0.06095" rpy="0 0 0"/>
       <axis xyz="0 0 1"/>
       <limit lower="-0.26" upper="0" effort="6"

Commit message: orient change

File: catchrobo_description/urdf/scara.urdf.xacro (robot description, xacro)
@@ -78,5 +78,5 @@
       <origin xyz="0.45 0 0" rpy="0 0 0"/>
       <axis xyz="0 0 1"/>
-      <limit lower="${-160*M_PI/180}" upper="${160*M_PI/180}" effort="6"
+      <limit lower="${-170*M_PI/180}" upper="${170*M_PI/180}" effort="6"
               velocity="5" acceleration="5"/>
     </joint>

Commit message: start error

File: catchrobo_description/urdf/scara.urdf.xacro (robot description, xacro)
@@ -52,9 +52,9 @@
       <axis xyz="0 0 1"/>
       <xacro:if value="${field=='blue'}">
-        <limit lower="${-90*M_PI/180}" upper="${160*M_PI/180}" effort="6"
+        <limit lower="${-30*M_PI/180}" upper="${160*M_PI/180}" effort="6"
               velocity="5" acceleration="5"/>
       </xacro:if>
       <xacro:if value="${field=='red'}">
-        <limit lower="${-160*M_PI/180}" upper="${90*M_PI/180}" effort="6"
+        <limit lower="${-160*M_PI/180}" upper="${30*M_PI/180}" effort="6"
               velocity="5" acceleration="5"/>
       </xacro:if>
