Commit message: hardware_update

File: catchrobo_description/urdf/base.urdf.xacro (robot description, xacro)
@@ -83,21 +83,59 @@
       </visual>
     </link>
-    <joint name="base/entry_prohibited_area" type="fixed">
+    <joint name="base/entry_prohibited_area_1" type="fixed">
       <parent link="base/base_link"/>
-      <child link="base/entry_prohibited_area"/>
+      <child link="base/entry_prohibited_area_1"/>
       <xacro:if value="${field=='blue'}">
-        <origin xyz="0.2 0.7 0.4" rpy="0 0 0"/>
+        <origin xyz="0.2 0.7 0.2" rpy="0 0 0"/>
       </xacro:if>
       <xacro:if value="${field=='red'}">
-        <origin xyz="-0.2 0.7 0.4" rpy="0 0 0"/>
+        <origin xyz="-0.2 0.7 0.2" rpy="0 0 0"/>
       </xacro:if>
     </joint>
-    <link name="base/entry_prohibited_area">
+    <link name="base/entry_prohibited_area_1">
       <visual>
         <geometry>
-          <box size="0.1 2.0 0.8"/>
+          <box size="0.1 2.0 0.4"/>
         </geometry>
         <origin xyz="0 0 0" rpy="0 0 0"/>
-        <material name="entry_prohibited_area"/>
+        <material name="entry_prohibited_area_1"/>
+      </visual>
+    </link>
+    <joint name="base/entry_prohibited_area_2" type="fixed">
+      <parent link="base/base_link"/>
+      <child link="base/entry_prohibited_area_2"/>
+      <xacro:if value="${field=='blue'}">
+        <origin xyz="-0.6 1.1 0.2" rpy="0 0 0"/>
+      </xacro:if>
+      <xacro:if value="${field=='red'}">
+        <origin xyz="0.6 1.1 0.2" rpy="0 0 0"/>
+      </xacro:if>
+    </joint>
+    <link name="base/entry_prohibited_area_2">
+      <visual>
+        <geometry>
+          <box size="2.0 0.1 0.4"/>
+        </geometry>
+        <origin xyz="0 0 0" rpy="0 0 0"/>
+        <material name="entry_prohibited_area_2"/>
+      </visual>
+    </link>
+    <joint name="base/entry_prohibited_area_3" type="fixed">
+      <parent link="base/base_link"/>
+      <child link="base/entry_prohibited_area_3"/>
+      <xacro:if value="${field=='blue'}">
+        <origin xyz="-0.6 -0.2 0.2" rpy="0 0 0"/>
+      </xacro:if>
+      <xacro:if value="${field=='red'}">
+        <origin xyz="0.6 -0.2 0.2" rpy="0 0 0"/>
+      </xacro:if>
+    </joint>
+    <link name="base/entry_prohibited_area_3">
+      <visual>
+        <geometry>
+          <box size="2.0 0.1 0.4"/>
+        </geometry>
+        <origin xyz="0 0 0" rpy="0 0 0"/>
+        <material name="entry_prohibited_area_3"/>
       </visual>
     </link>

Commit message: hadware_update

File: catchrobo_description/urdf/base.urdf.xacro (robot description, xacro)
@@ -99,5 +99,5 @@
         </geometry>
         <origin xyz="0 0 0" rpy="0 0 0"/>
-        <material name="entry_prohibited_area_1"/>
+        <material name="grey"/>
       </visual>
     </link>
@@ -118,5 +118,5 @@
         </geometry>
         <origin xyz="0 0 0" rpy="0 0 0"/>
-        <material name="entry_prohibited_area_2"/>
+        <material name="grey"/>
       </visual>
     </link>
@@ -137,5 +137,24 @@
         </geometry>
         <origin xyz="0 0 0" rpy="0 0 0"/>
-        <material name="entry_prohibited_area_3"/>
+        <material name="grey"/>
+      </visual>
+    </link>
+    <joint name="base/weight_box" type="fixed">
+      <parent link="base/base_link"/>
+      <child link="base/weight_box"/>
+      <xacro:if value="${field=='blue'}">
+        <origin xyz="-1.2 0.25 0.125" rpy="0 0 0"/>
+      </xacro:if>
+      <xacro:if value="${field=='red'}">
+        <origin xyz="1.2 0.25 0.125" rpy="0 0 0"/>
+      </xacro:if>
+    </joint>
+    <link name="base/weight_box">
+      <visual>
+        <geometry>
+          <box size="0.4 0.3 0.25"/>
+        </geometry>
+        <origin xyz="0 0 0" rpy="0 0 0"/>
+        <material name="grey"/>
       </visual>
     </link>

Commit message: joint limits and protection wall mesh update

File: catchrobo_description/urdf/base.urdf.xacro (robot description, xacro)
@@ -68,8 +68,8 @@
       <child link="base/pc"/>
       <xacro:if value="${field=='blue'}">
-        <origin xyz="-0.85 0 0.12" rpy="0 0 0"/>
+        <origin xyz="-0.85 0 0.15" rpy="0 0 0"/>
       </xacro:if>
       <xacro:if value="${field=='red'}">
-        <origin xyz="0.85 0 0.12" rpy="0 0 0"/>
+        <origin xyz="0.85 0 0.15" rpy="0 0 0"/>
       </xacro:if>
     </joint>
@@ -77,8 +77,8 @@
       <visual>
         <geometry>
-          <box size="0.25 0.4 0.24"/>
+          <box size="0.25 0.4 0.3"/>
         </geometry>
         <origin xyz="0 0 0" rpy="0 0 0"/>
-        <material name="grey"/>
+        <material name="clear_grey"/>
       </visual>
     </link>
@@ -87,8 +87,8 @@
       <child link="base/entry_prohibited_area_1"/>
       <xacro:if value="${field=='blue'}">
-        <origin xyz="0.2 0.7 0.2" rpy="0 0 0"/>
+        <origin xyz="0.2 0.45 0.25" rpy="0 0 0"/>
       </xacro:if>
       <xacro:if value="${field=='red'}">
-        <origin xyz="-0.2 0.7 0.2" rpy="0 0 0"/>
+        <origin xyz="-0.2 0.45 0.25" rpy="0 0 0"/>
       </xacro:if>
     </joint>
@@ -96,8 +96,8 @@
       <visual>
         <geometry>
-          <box size="0.1 2.0 0.4"/>
+          <box size="0.1 1.3 0.5"/>
         </geometry>
         <origin xyz="0 0 0" rpy="0 0 0"/>
-        <material name="grey"/>
+        <material name="clear_grey"/>
       </visual>
     </link>
@@ -106,8 +106,8 @@
       <child link="base/entry_prohibited_area_2"/>
       <xacro:if value="${field=='blue'}">
-        <origin xyz="-0.6 1.1 0.2" rpy="0 0 0"/>
+        <origin xyz="-0.25 1.05 0.25" rpy="0 0 0"/>
       </xacro:if>
       <xacro:if value="${field=='red'}">
-        <origin xyz="0.6 1.1 0.2" rpy="0 0 0"/>
+        <origin xyz="0.25 1.05 0.25" rpy="0 0 0"/>
       </xacro:if>
     </joint>
@@ -115,8 +115,8 @@
       <visual>
         <geometry>
-          <box size="2.0 0.1 0.4"/>
+          <box size="1.0 0.1 0.5"/>
         </geometry>
         <origin xyz="0 0 0" rpy="0 0 0"/>
-        <material name="grey"/>
+        <material name="clear_grey"/>
       </visual>
     </link>
@@ -125,8 +125,8 @@
       <child link="base/entry_prohibited_area_3"/>
       <xacro:if value="${field=='blue'}">
-        <origin xyz="-0.6 -0.2 0.2" rpy="0 0 0"/>
+        <origin xyz="-0.25 -0.15 0.25" rpy="0 0 0"/>
       </xacro:if>
       <xacro:if value="${field=='red'}">
-        <origin xyz="0.6 -0.2 0.2" rpy="0 0 0"/>
+        <origin xyz="0.25 -0.15 0.25" rpy="0 0 0"/>
       </xacro:if>
     </joint>
@@ -134,10 +134,11 @@
       <visual>
         <geometry>
-          <box size="2.0 0.1 0.4"/>
+          <box size="1.0 0.1 0.5"/>
         </geometry>
         <origin xyz="0 0 0" rpy="0 0 0"/>
-        <material name="grey"/>
+        <material name="clear_grey"/>
       </visual>
     </link>
+    <!--
     <joint name="base/weight_box" type="fixed">
       <parent link="base/base_link"/>
@@ -156,7 +157,8 @@
         </geometry>
         <origin xyz="0 0 0" rpy="0 0 0"/>
-        <material name="grey"/>
+        <material name="clear_grey"/>
       </visual>
     </link>
+    -->
   </xacro:macro>
 </robot>

File: catchrobo_description/urdf/materials.xacro (robot description, xacro)
@@ -34,3 +34,6 @@
     <color rgba="0.5 0.5 0.5 0.1"/>
   </material>
+  <material name="clear_grey">
+    <color rgba="0.2 0.2 0.2 0.5"/>
+  </material>
 </robot>

Commit message: scara mesh&urdf update

File: catchrobo_description/urdf/base.urdf.xacro (robot description, xacro)
@@ -68,8 +68,8 @@
       <child link="base/pc"/>
       <xacro:if value="${field=='blue'}">
-        <origin xyz="-0.85 0 0.15" rpy="0 0 0"/>
+        <origin xyz="-0.85 0 0.125" rpy="0 0 0"/>
       </xacro:if>
       <xacro:if value="${field=='red'}">
-        <origin xyz="0.85 0 0.15" rpy="0 0 0"/>
+        <origin xyz="0.85 0 0.125" rpy="0 0 0"/>
       </xacro:if>
     </joint>
@@ -77,5 +77,5 @@
       <visual>
         <geometry>
-          <box size="0.25 0.4 0.3"/>
+          <box size="0.25 0.4 0.25"/>
         </geometry>
         <origin xyz="0 0 0" rpy="0 0 0"/>

File: catchrobo_description/urdf/scara.urdf.xacro (robot description, xacro)
@@ -28,5 +28,5 @@
       <parent link="${prefix}arm/link0"/>
       <child link="${prefix}arm/link1"/>
-      <origin xyz="0 0 0.4325" rpy="0 0 0"/>
+      <origin xyz="0 0 0.3375" rpy="0 0 0"/>
       <axis xyz="0 0 1"/>
       <limit lower="${-160*M_PI/180}" upper="${160*M_PI/180}" effort="6"
@@ -99,5 +99,5 @@
       <origin xyz="0 0 -0.03295" rpy="0 0 0"/>
       <axis xyz="0 0 1"/>
-      <limit lower="-0.35" upper="0" effort="6"
+      <limit lower="-0.26" upper="0" effort="6"
               velocity="5" acceleration="5"/>
     </joint>

Commit message: robot position changed, link0 mesh bolded

File: catchrobo_description/urdf/base.urdf.xacro (robot description, xacro)
@@ -46,8 +46,8 @@
       <child link="base/robot_tip"/>
       <xacro:if value="${field=='blue'}">
-        <origin xyz="-0.795 0.390 0.0044" rpy="0 0 0"/>
+        <origin xyz="-0.795 0.350 0.0044" rpy="0 0 0"/>
       </xacro:if>
       <xacro:if value="${field=='red'}">
-        <origin xyz="0.795 0.390 0.0044" rpy="0 0 ${180*M_PI/180}"/>
+        <origin xyz="0.795 0.350 0.0044" rpy="0 0 ${180*M_PI/180}"/>
       </xacro:if>
     </joint>
@@ -125,8 +125,8 @@
       <child link="base/entry_prohibited_area_3"/>
       <xacro:if value="${field=='blue'}">
-        <origin xyz="-0.25 -0.15 0.25" rpy="0 0 0"/>
+        <origin xyz="-0.25 -0.20 0.25" rpy="0 0 0"/>
       </xacro:if>
       <xacro:if value="${field=='red'}">
-        <origin xyz="0.25 -0.15 0.25" rpy="0 0 0"/>
+        <origin xyz="0.25 -0.20 0.25" rpy="0 0 0"/>
       </xacro:if>
     </joint>
@@ -140,13 +140,12 @@
       </visual>
     </link>
-    <!--
     <joint name="base/weight_box" type="fixed">
       <parent link="base/base_link"/>
       <child link="base/weight_box"/>
       <xacro:if value="${field=='blue'}">
-        <origin xyz="-1.2 0.25 0.125" rpy="0 0 0"/>
+        <origin xyz="-1.2 0.25 0.15" rpy="0 0 0"/>
       </xacro:if>
       <xacro:if value="${field=='red'}">
-        <origin xyz="1.2 0.25 0.125" rpy="0 0 0"/>
+        <origin xyz="1.2 0.25 0.15" rpy="0 0 0"/>
       </xacro:if>
     </joint>
@@ -154,5 +153,5 @@
       <visual>
         <geometry>
-          <box size="0.4 0.3 0.25"/>
+          <box size="0.4 0.3 0.3"/>
         </geometry>
         <origin xyz="0 0 0" rpy="0 0 0"/>
@@ -160,5 +159,4 @@
       </visual>
     </link>
-    -->
   </xacro:macro>
 </robot>

File: catchrobo_description/urdf/scara.urdf.xacro (robot description, xacro)
@@ -21,5 +21,5 @@
       <collision>
         <geometry>
-          <mesh filename="package://catchrobo_description/mesh/scara/collision/link0.stl" scale="${collision_mesh_scale}"/>
+          <mesh filename="package://catchrobo_description/mesh/scara/collision/link0_bold.stl" scale="${collision_mesh_scale}"/>
         </geometry>
       </collision>

Commit message: add shootingbox

File: catchrobo_description/urdf/base.urdf.xacro (robot description, xacro)
@@ -46,8 +46,8 @@
       <child link="base/robot_tip"/>
       <xacro:if value="${field=='blue'}">
-        <origin xyz="-0.795 0.390 0.0044" rpy="0 0 0"/>
+        <origin xyz="-0.795 0.350 0.0044" rpy="0 0 0"/>
       </xacro:if>
       <xacro:if value="${field=='red'}">
-        <origin xyz="0.795 0.390 0.0044" rpy="0 0 ${180*M_PI/180}"/>
+        <origin xyz="0.795 0.350 0.0044" rpy="0 0 ${180*M_PI/180}"/>
       </xacro:if>
     </joint>
@@ -68,8 +68,8 @@
       <child link="base/pc"/>
       <xacro:if value="${field=='blue'}">
-        <origin xyz="-0.85 0 0.12" rpy="0 0 0"/>
+        <origin xyz="-0.85 0 0.125" rpy="0 0 0"/>
       </xacro:if>
       <xacro:if value="${field=='red'}">
-        <origin xyz="0.85 0 0.12" rpy="0 0 0"/>
+        <origin xyz="0.85 0 0.125" rpy="0 0 0"/>
       </xacro:if>
     </joint>
@@ -77,27 +77,84 @@
       <visual>
         <geometry>
-          <box size="0.25 0.4 0.24"/>
+          <box size="0.25 0.4 0.25"/>
         </geometry>
         <origin xyz="0 0 0" rpy="0 0 0"/>
-        <material name="grey"/>
+        <material name="clear_grey"/>
       </visual>
     </link>
-    <joint name="base/entry_prohibited_area" type="fixed">
+    <joint name="base/entry_prohibited_area_1" type="fixed">
       <parent link="base/base_link"/>
-      <child link="base/entry_prohibited_area"/>
+      <child link="base/entry_prohibited_area_1"/>
       <xacro:if value="${field=='blue'}">
-        <origin xyz="0.2 0.7 0.4" rpy="0 0 0"/>
+        <origin xyz="0.2 0.45 0.25" rpy="0 0 0"/>
       </xacro:if>
       <xacro:if value="${field=='red'}">
-        <origin xyz="-0.2 0.7 0.4" rpy="0 0 0"/>
+        <origin xyz="-0.2 0.45 0.25" rpy="0 0 0"/>
       </xacro:if>
     </joint>
-    <link name="base/entry_prohibited_area">
+    <link name="base/entry_prohibited_area_1">
       <visual>
         <geometry>
-          <box size="0.1 2.0 0.8"/>
+          <box size="0.1 1.3 0.5"/>
         </geometry>
         <origin xyz="0 0 0" rpy="0 0 0"/>
-        <material name="entry_prohibited_area"/>
+        <material name="clear_grey"/>
+      </visual>
+    </link>
+    <joint name="base/entry_prohibited_area_2" type="fixed">
+      <parent link="base/base_link"/>
+      <child link="base/entry_prohibited_area_2"/>
+      <xacro:if value="${field=='blue'}">
+        <origin xyz="-0.25 1.05 0.25" rpy="0 0 0"/>
+      </xacro:if>
+      <xacro:if value="${field=='red'}">
+        <origin xyz="0.25 1.05 0.25" rpy="0 0 0"/>
+      </xacro:if>
+    </joint>
+    <link name="base/entry_prohibited_area_2">
+      <visual>
+        <geometry>
+          <box size="1.0 0.1 0.5"/>
+        </geometry>
+        <origin xyz="0 0 0" rpy="0 0 0"/>
+        <material name="clear_grey"/>
+      </visual>
+    </link>
+    <joint name="base/entry_prohibited_area_3" type="fixed">
+      <parent link="base/base_link"/>
+      <child link="base/entry_prohibited_area_3"/>
+      <xacro:if value="${field=='blue'}">
+        <origin xyz="-0.25 -0.20 0.25" rpy="0 0 0"/>
+      </xacro:if>
+      <xacro:if value="${field=='red'}">
+        <origin xyz="0.25 -0.20 0.25" rpy="0 0 0"/>
+      </xacro:if>
+    </joint>
+    <link name="base/entry_prohibited_area_3">
+      <visual>
+        <geometry>
+          <box size="1.0 0.1 0.5"/>
+        </geometry>
+        <origin xyz="0 0 0" rpy="0 0 0"/>
+        <material name="clear_grey"/>
+      </visual>
+    </link>
+    <joint name="base/weight_box" type="fixed">
+      <parent link="base/base_link"/>
+      <child link="base/weight_box"/>
+      <xacro:if value="${field=='blue'}">
+        <origin xyz="-1.2 0.25 0.15" rpy="0 0 0"/>
+      </xacro:if>
+      <xacro:if value="${field=='red'}">
+        <origin xyz="1.2 0.25 0.15" rpy="0 0 0"/>
+      </xacro:if>
+    </joint>
+    <link name="base/weight_box">
+      <visual>
+        <geometry>
+          <box size="0.4 0.3 0.3"/>
+        </geometry>
+        <origin xyz="0 0 0" rpy="0 0 0"/>
+        <material name="clear_grey"/>
       </visual>
     </link>

File: catchrobo_description/urdf/scara.urdf.xacro (robot description, xacro)
@@ -21,5 +21,5 @@
       <collision>
         <geometry>
-          <mesh filename="package://catchrobo_description/mesh/scara/collision/link0.stl" scale="${collision_mesh_scale}"/>
+          <mesh filename="package://catchrobo_description/mesh/scara/collision/link0_bold.stl" scale="${collision_mesh_scale}"/>
         </geometry>
       </collision>
@@ -28,5 +28,5 @@
       <parent link="${prefix}arm/link0"/>
       <child link="${prefix}arm/link1"/>
-      <origin xyz="0 0 0.3175" rpy="0 0 0"/>
+      <origin xyz="0 0 0.3875" rpy="0 0 0"/>
       <axis xyz="0 0 1"/>
       <limit lower="${-160*M_PI/180}" upper="${160*M_PI/180}" effort="6"
@@ -49,5 +49,5 @@
       <parent link="${prefix}arm/link1"/>
       <child link="${prefix}arm/link2"/>
-      <origin xyz="0.45 0 0.043" rpy="0 0 0"/>
+      <origin xyz="0.45 0 0.04308" rpy="0 0 0"/>
       <axis xyz="0 0 1"/>
       <xacro:if value="${field=='blue'}">
@@ -97,7 +97,7 @@
       <parent link="${prefix}arm/link3"/>
       <child link="${prefix}arm/link4"/>
-      <origin xyz="0 0 -0.0335" rpy="0 0 0"/>
+      <origin xyz="0 0 -0.06095" rpy="0 0 0"/>
       <axis xyz="0 0 1"/>
-      <limit lower="-0.25" upper="0" effort="6"
+      <limit lower="-0.26" upper="0" effort="6"
               velocity="5" acceleration="5"/>
     </joint>

Commit message: update

File: catchrobo_description/urdf/base.urdf.xacro (robot description, xacro)
@@ -106,8 +106,8 @@
       <child link="base/entry_prohibited_area_2"/>
       <xacro:if value="${field=='blue'}">
-        <origin xyz="-0.25 1.05 0.25" rpy="0 0 0"/>
+        <origin xyz="-0.25 1.2 0.25" rpy="0 0 0"/>
       </xacro:if>
       <xacro:if value="${field=='red'}">
-        <origin xyz="0.25 1.05 0.25" rpy="0 0 0"/>
+        <origin xyz="0.25 1.2 0.25" rpy="0 0 0"/>
       </xacro:if>
     </joint>

Commit message: obstacle

File: catchrobo_description/urdf/base.urdf.xacro (robot description, xacro)
@@ -114,8 +114,8 @@
       <child link="base/entry_prohibited_area_2"/>
       <xacro:if value="${field=='blue'}">
-        <origin xyz="-0.25 1.2 0.25" rpy="0 0 0"/>
+        <origin xyz="-0.25 1.1 0.25" rpy="0 0 0"/>
       </xacro:if>
       <xacro:if value="${field=='red'}">
-        <origin xyz="0.25 1.2 0.25" rpy="0 0 0"/>
+        <origin xyz="0.25 1.1 0.25" rpy="0 0 0"/>
       </xacro:if>
     </joint>
@@ -123,5 +123,5 @@
       <visual>
         <geometry>
-          <box size="1.0 0.1 0.5"/>
+          <box size="3.0 0.1 0.5"/>
         </geometry>
         <origin xyz="0 0 0" rpy="0 0 0"/>

Commit message: testrun touzitu

File: catchrobo_description/urdf/base.urdf.xacro (robot description, xacro)
@@ -114,8 +114,8 @@
       <child link="base/entry_prohibited_area_2"/>
       <xacro:if value="${field=='blue'}">
-        <origin xyz="-0.25 1.1 0.25" rpy="0 0 0"/>
+        <origin xyz="-0.25 1.2 0.25" rpy="0 0 0"/>
       </xacro:if>
       <xacro:if value="${field=='red'}">
-        <origin xyz="0.25 1.1 0.25" rpy="0 0 0"/>
+        <origin xyz="0.25 1.2 0.25" rpy="0 0 0"/>
       </xacro:if>
     </joint>
@@ -148,4 +148,23 @@
       </visual>
     </link>
+    <!-- <joint name="base/entry_prohibited_area_4" type="fixed">
+      <parent link="base/base_link"/>
+      <child link="base/entry_prohibited_area_4"/>
+      <xacro:if value="${field=='blue'}">
+        <origin xyz="-1.0 0.5 0.1" rpy="0 0 0"/>
+      </xacro:if>
+      <xacro:if value="${field=='red'}">
+        <origin xyz="1.0 0.5 0.1" rpy="0 0 0"/>
+      </xacro:if>
+    </joint>
+    <link name="base/entry_prohibited_area_4">
+      <visual>
+        <geometry>
+          <box size="0.4 0.3 0.2"/>
+        </geometry>
+        <origin xyz="0 0 0" rpy="0 0 0"/>
+        <material name="clear_grey"/>
+      </visual>
+    </link> -->
     <joint name="base/weight_box" type="fixed">
       <parent link="base/base_link"/>
