Commit message: plan is bad

File: catchrobo_description/robots/catchrobo.urdf.xacro (robot description, xacro)
@@ -2,11 +2,11 @@
 <robot name="catchrobo" xmlns:xacro="http://ros.org/wiki/xacro">
   <!-- Dependencies -->
-  <xacro:include filename="$(find catchrobo_description)/urdf/materials.xacro"/>
-  <xacro:include filename="$(find catchrobo_description)/urdf/common.xacro"/>
-  <xacro:include filename="$(find catchrobo_description)/urdf/base.urdf.xacro"/>
-  <xacro:include filename="$(find catchrobo_description)/urdf/arm.urdf.xacro"/>
-  <xacro:include filename="$(find catchrobo_description)/urdf/gripper.urdf.xacro"/>
+  <xacro:include filename="$(find catchrobo_description)/urdf/materials.xacro" />
+  <xacro:include filename="$(find catchrobo_description)/urdf/common.xacro" />
+  <xacro:include filename="$(find catchrobo_description)/urdf/base.urdf.xacro" />
+  <xacro:include filename="$(find catchrobo_description)/urdf/arm.urdf.xacro" />
+  <xacro:include filename="$(find catchrobo_description)/urdf/gripper.urdf.xacro" />
   <!-- Link & Joint -->
-  <link name="world"/>
+  <link name="world" />
   <xacro:base parent="world">
     <origin xyz="0 0 0" rpy="0 0 0" />

Commit message: set collision to bisco

File: catchrobo_description/robots/catchrobo.urdf.xacro (robot description, xacro)
@@ -1,4 +1,6 @@
 <?xml version="1.0"?>
 <robot name="catchrobo" xmlns:xacro="http://ros.org/wiki/xacro">
+  <xacro:arg name="field" default="" />
+  <xacro:property name="field" value="$(arg field)" />
   <!-- Dependencies -->
   <xacro:include filename="$(find catchrobo_description)/urdf/materials.xacro" />
@@ -13,5 +15,10 @@
   </xacro:base>
   <xacro:arm prefix="" parent="base/link_tip">
-    <origin xyz="0 0 0" rpy="0 0 0" />
+    <xacro:if value="${field=='blue'}">
+      <origin xyz="0 0 0.08" rpy="0 0 ${-90*M_PI/180}" />
+    </xacro:if>
+    <xacro:if value="${field=='red'}">
+      <origin xyz="0 0 0" rpy="0 0 ${90*M_PI/180}" />
+    </xacro:if>
   </xacro:arm>
   <xacro:gripper prefix="" parent="arm/link_tip">

File: catchrobo_description/urdf/arm.urdf.xacro (robot description, xacro)
@@ -2,6 +2,6 @@
 <robot xmlns:xacro="http://ros.org/wiki/xacro">
   <!-- Constants -->
-  <xacro:property name="visual_mesh_scale" value="1.0 1.0 1.0"/>
-  <xacro:property name="collision_mesh_scale" value="1.0 1.0 1.0"/>
+  <xacro:property name="visual_mesh_scale" value="1.0 1.0 1.0" />
+  <xacro:property name="collision_mesh_scale" value="1.0 1.0 1.0" />
   <!-- Link & Joint -->
   <xacro:macro name="arm" params="prefix parent *joint_origin">
@@ -14,125 +14,127 @@
       <visual>
         <geometry>
-          <mesh filename="package://catchrobo_description/mesh/arm/link0.stl" scale="${visual_mesh_scale}"/>
+          <mesh filename="package://catchrobo_description/mesh/arm/link0.stl" scale="${visual_mesh_scale}" />
         </geometry>
-        <material name="orange"/>
+        <material name="orange" />
       </visual>
       <collision>
         <geometry>
-          <mesh filename="package://catchrobo_description/mesh/arm/link0.stl" scale="${collision_mesh_scale}"/>
+          <mesh filename="package://catchrobo_description/mesh/arm/link0.stl" scale="${collision_mesh_scale}" />
         </geometry>
       </collision>
     </link>
     <joint name="${prefix}arm/joint1" type="revolute">
-      <parent link="${prefix}arm/link0"/>
-      <child link="${prefix}arm/link1"/>
-      <origin xyz="0 0 0.08" rpy="0 0 0"/>
-      <axis xyz="0 0 1"/>
-      <limit lower="${-90*M_PI/180}" upper="${90*M_PI/180}" effort="6"
-              velocity="5" acceleration="5"/>
+      <parent link="${prefix}arm/link0" />
+      <child link="${prefix}arm/link1" />
+      <origin xyz="0 0 0.08" rpy="0 0 0" />
+      <axis xyz="0 0 1" />
+      <limit lower="${-150*M_PI/180}" upper="${150*M_PI/180}" effort="6" velocity="5" acceleration="5" />
     </joint>
     <link name="${prefix}arm/link1">
       <visual>
         <geometry>
-          <mesh filename="package://catchrobo_description/mesh/arm/link1.stl" scale="${visual_mesh_scale}"/>
+          <mesh filename="package://catchrobo_description/mesh/arm/link1.stl" scale="${visual_mesh_scale}" />
         </geometry>
-        <material name="orange"/>
+        <material name="orange" />
       </visual>
       <collision>
         <geometry>
-          <mesh filename="package://catchrobo_description/mesh/arm/link1.stl" scale="${collision_mesh_scale}"/>
+          <mesh filename="package://catchrobo_description/mesh/arm/link1.stl" scale="${collision_mesh_scale}" />
         </geometry>
       </collision>
     </link>
     <joint name="${prefix}arm/joint2" type="revolute">
-      <parent link="${prefix}arm/link1"/>
-      <child link="${prefix}arm/link2"/>
-      <origin xyz="0 0 0.08" rpy="${90*M_PI/180} 0 ${90*M_PI/180}"/>
-      <axis xyz="0 0 1"/>
-      <limit lower="${-90*M_PI/180}" upper="${90*M_PI/180}" effort="6"
-              velocity="5" acceleration="5"/>
+      <parent link="${prefix}arm/link1" />
+      <child link="${prefix}arm/link2" />
+      <origin xyz="0 0 0.08" rpy="${90*M_PI/180} 0 ${90*M_PI/180}" />
+      <axis xyz="0 0 1" />
+      <limit lower="${-90*M_PI/180}" upper="${90*M_PI/180}" effort="6" velocity="5" acceleration="5" />
     </joint>
     <link name="${prefix}arm/link2">
       <visual>
         <geometry>
-          <mesh filename="package://catchrobo_description/mesh/arm/link2.stl" scale="${visual_mesh_scale}"/>
+          <mesh filename="package://catchrobo_description/mesh/arm/link2.stl" scale="${visual_mesh_scale}" />
         </geometry>
-        <material name="orange"/>
+        <material name="orange" />
       </visual>
       <collision>
         <geometry>
-          <mesh filename="package://catchrobo_description/mesh/arm/link2.stl" scale="${collision_mesh_scale}"/>
+          <mesh filename="package://catchrobo_description/mesh/arm/link2.stl" scale="${collision_mesh_scale}" />
         </geometry>
       </collision>
     </link>
     <joint name="${prefix}arm/joint3" type="revolute">
-      <parent link="${prefix}arm/link2"/>
-      <child link="${prefix}arm/link3"/>
-      <origin xyz="0 0.4 0" rpy="0 0 0"/>
-      <axis xyz="0 0 1"/>
-      <limit lower="${-135*M_PI/180}" upper="${135*M_PI/180}" effort="6"
-              velocity="5" acceleration="5"/>
+      <parent link="${prefix}arm/link2" />
+      <child link="${prefix}arm/link3" />
+      <origin xyz="0 0.45 0" rpy="0 0 0" />
+      <axis xyz="0 0 1" />
+      <limit lower="${-160*M_PI/180}" upper="0" effort="6" velocity="5" acceleration="5" />
     </joint>
     <link name="${prefix}arm/link3">
       <visual>
         <geometry>
-          <mesh filename="package://catchrobo_description/mesh/arm/link3.stl" scale="${visual_mesh_scale}"/>
+          <mesh filename="package://catchrobo_description/mesh/arm/link3.stl" scale="${visual_mesh_scale}" />
         </geometry>
-        <material name="orange"/>
+        <material name="orange" />
       </visual>
       <collision>
         <geometry>
-          <mesh filename="package://catchrobo_description/mesh/arm/link3.stl" scale="${collision_mesh_scale}"/>
+          <mesh filename="package://catchrobo_description/mesh/arm/link3.stl" scale="${collision_mesh_scale}" />
         </geometry>
       </collision>
     </link>
     <joint name="${prefix}arm/joint4" type="revolute">
-      <parent link="${prefix}arm/link3"/>
-      <child link="${prefix}arm/link4"/>
-      <origin xyz="0 0.4 0" rpy="0 0 0"/>
-      <axis xyz="0 0 1"/>
-      <limit lower="${-90*M_PI/180}" upper="${90*M_PI/180}" effort="6"
-              velocity="5" acceleration="5"/>
+      <parent link="${prefix}arm/link3" />
+      <child link="${prefix}arm/link4" />
+      <origin xyz="0 0.45 0" rpy="0 0 0" />
+      <axis xyz="0 0 1" />
+      <limit lower="${-90*M_PI/180}" upper="${90*M_PI/180}" effort="6" velocity="5" acceleration="5" />
     </joint>
     <link name="${prefix}arm/link4">
       <visual>
         <geometry>
-          <mesh filename="package://catchrobo_description/mesh/arm/link4.stl" scale="${visual_mesh_scale}"/>
+          <mesh filename="package://catchrobo_description/mesh/arm/link4.stl" scale="${visual_mesh_scale}" />
         </geometry>
-        <material name="orange"/>
+        <material name="orange" />
       </visual>
       <collision>
         <geometry>
-          <mesh filename="package://catchrobo_description/mesh/arm/link4.stl" scale="${collision_mesh_scale}"/>
+          <mesh filename="package://catchrobo_description/mesh/arm/link4.stl" scale="${collision_mesh_scale}" />
         </geometry>
       </collision>
     </link>
     <joint name="${prefix}arm/joint5" type="revolute">
-      <parent link="${prefix}arm/link4"/>
-      <child link="${prefix}arm/link5"/>
-      <origin xyz="0 0.04 0" rpy="${-90*M_PI/180} 0 0"/>
-      <axis xyz="0 0 1"/>
-      <limit lower="${-180*M_PI/180}" upper="${180*M_PI/180}" effort="6"
-              velocity="5" acceleration="5"/>
+      <parent link="${prefix}arm/link4" />
+      <child link="${prefix}arm/link5" />
+      <origin xyz="0 0.04 0" rpy="${-90*M_PI/180} 0 0" />
+      <axis xyz="0 0 1" />
+      <limit lower="${-150*M_PI/180}" upper="${150*M_PI/180}" effort="6" velocity="5" acceleration="5" />
     </joint>
     <link name="${prefix}arm/link5">
       <visual>
         <geometry>
-          <mesh filename="package://catchrobo_description/mesh/arm/link5.stl" scale="${visual_mesh_scale}"/>
+          <mesh filename="package://catchrobo_description/mesh/arm/link5.stl" scale="${visual_mesh_scale}" />
         </geometry>
-        <material name="orange"/>
+        <material name="orange" />
       </visual>
       <collision>
         <geometry>
-          <mesh filename="package://catchrobo_description/mesh/arm/link5.stl" scale="${collision_mesh_scale}"/>
+          <mesh filename="package://catchrobo_description/mesh/arm/link5.stl" scale="${collision_mesh_scale}" />
         </geometry>
       </collision>
     </link>
     <joint name="${prefix}arm/joint_tip" type="fixed">
-      <parent link="${prefix}arm/link5"/>
-      <child link="${prefix}arm/link_tip"/>
-      <origin xyz="0 0 0.02" rpy="0 0 0"/>
+      <parent link="${prefix}arm/link5" />
+      <child link="${prefix}arm/link_tip" />
+      <origin xyz="0 0 0.02" rpy="0 0 0" />
     </joint>
-    <link name="${prefix}arm/link_tip"/>
+    <link name="${prefix}arm/link_tip" />
+    <!-- Transmissions -->
+    <!-- <xacro:include filename="$(find catchrobo_description)/urdf/arm.transmission.xacro" />
+    <arm_simple_transmission id="1" reduction="1.0" />
+    <arm_simple_transmission id="2" reduction="1.0" />
+    <arm_simple_transmission id="3" reduction="1.0" />
+    <arm_simple_transmission id="4" reduction="1.0" />
+    <arm_simple_transmission id="5" reduction="1.0" /> -->
   </xacro:macro>
 </robot>

File: catchrobo_description/urdf/base.urdf.xacro (robot description, xacro)
@@ -2,27 +2,27 @@
 <robot xmlns:xacro="http://ros.org/wiki/xacro">
   <!-- Field Side Parameters-->
-  <xacro:arg name="field" default=""/>
+  <xacro:arg name="field" default="" />
   <xacro:property name="field" value="$(arg field)" />
   <!-- Constants -->
-  <xacro:property name="visual_mesh_scale" value="1.0 1.0 1.0"/>
-  <xacro:property name="collision_mesh_scale" value="1.0 1.0 1.0"/>
+  <xacro:property name="visual_mesh_scale" value="1.0 1.0 1.0" />
+  <xacro:property name="collision_mesh_scale" value="1.0 1.0 1.0" />
   <!-- Link & Joint -->
   <xacro:macro name="base" params="parent *joint_origin">
     <joint name="base/root" type="fixed">
-      <xacro:insert_block name="joint_origin"/>
-      <parent link="${parent}"/>
-      <child link="base/base_link"/>
+      <xacro:insert_block name="joint_origin" />
+      <parent link="${parent}" />
+      <child link="base/base_link" />
     </joint>
-    <link name="base/base_link">
+    <!-- <link name="base/base_link">
       <xacro:if value="${field=='blue'}">
         <visual>
           <geometry>
-            <mesh filename="package://catchrobo_description/mesh/base/base_blue.stl" scale="${visual_mesh_scale}"/>
+            <mesh filename="package://catchrobo_description/mesh/base/base_blue.stl" scale="${visual_mesh_scale}" />
           </geometry>
-          <material name="white"/>
+          <material name="white" />
         </visual>
         <collision>
           <geometry>
-            <mesh filename="package://catchrobo_description/mesh/base/base_blue.stl" scale="${collision_mesh_scale}"/>
+            <mesh filename="package://catchrobo_description/mesh/base/base_blue.stl" scale="${collision_mesh_scale}" />
           </geometry>
         </collision>
@@ -31,11 +31,39 @@
         <visual>
           <geometry>
-            <mesh filename="package://catchrobo_description/mesh/base/base_red.stl" scale="${visual_mesh_scale}"/>
+            <mesh filename="package://catchrobo_description/mesh/base/base_red.stl" scale="${visual_mesh_scale}" />
           </geometry>
-          <material name="white"/>
+          <material name="white" />
         </visual>
         <collision>
           <geometry>
-            <mesh filename="package://catchrobo_description/mesh/base/base_red.stl" scale="${collision_mesh_scale}"/>
+            <mesh filename="package://catchrobo_description/mesh/base/base_red.stl" scale="${collision_mesh_scale}" />
+          </geometry>
+        </collision>
+      </xacro:if>
+    </link> -->
+    <link name="base/base_link">
+      <xacro:if value="${field=='blue'}">
+        <visual>
+          <geometry>
+            <mesh filename="package://catchrobo_description/mesh/base/blue_side_without_bisco_re.stl.stl" scale="${visual_mesh_scale}" />
+          </geometry>
+          <material name="white" />
+        </visual>
+        <collision>
+          <geometry>
+            <mesh filename="package://catchrobo_description/mesh/base/blue_side_without_bisco_re.stl.stl" scale="${collision_mesh_scale}" />
+          </geometry>
+        </collision>
+      </xacro:if>
+      <xacro:if value="${field=='red'}">
+        <visual>
+          <geometry>
+            <mesh filename="package://catchrobo_description/mesh/base/red_side_without_bisco_re.stl" scale="${visual_mesh_scale}" />
+          </geometry>
+          <material name="white" />
+        </visual>
+        <collision>
+          <geometry>
+            <mesh filename="package://catchrobo_description/mesh/base/red_side_without_bisco_re.stl" scale="${collision_mesh_scale}" />
           </geometry>
         </collision>
@@ -43,14 +71,14 @@
     </link>
     <joint name="base/joint_tip" type="fixed">
-      <parent link="base/base_link"/>
-      <child link="base/link_tip"/>
+      <parent link="base/base_link" />
+      <child link="base/link_tip" />
       <xacro:if value="${field=='blue'}">
-        <origin xyz="-0.8 0.4 0.0044" rpy="0 0 0"/>
+        <origin xyz="-0.8 0.4 0.0044" rpy="0 0 0" />
       </xacro:if>
       <xacro:if value="${field=='red'}">
-        <origin xyz="0.8 0.4 0.0044" rpy="0 0 0"/>
+        <origin xyz="0.8 0.4 0.0044" rpy="0 0 0" />
       </xacro:if>
     </joint>
-    <link name="base/link_tip"/>
+    <link name="base/link_tip" />
   </xacro:macro>
 </robot>
