Commit message: mesh and urdf update

File: catchrobo_description/robots/catchrobo.urdf.xacro (robot description, xacro)
@@ -15,10 +15,5 @@
   </xacro:base>
   <xacro:arm prefix="" parent="base/link_tip">
-    <xacro:if value="${field=='blue'}">
-      <origin xyz="0 0 0.08" rpy="0 0 ${-90*M_PI/180}" />
-    </xacro:if>
-    <xacro:if value="${field=='red'}">
-      <origin xyz="0 0 0" rpy="0 0 ${90*M_PI/180}" />
-    </xacro:if>
+    <origin xyz="0 0 0" rpy="0 0 0" />
   </xacro:arm>
   <xacro:gripper prefix="" parent="arm/link_tip">

File: catchrobo_description/urdf/arm.urdf.xacro (robot description, xacro)
@@ -2,6 +2,6 @@
 <robot xmlns:xacro="http://ros.org/wiki/xacro">
   <!-- Constants -->
-  <xacro:property name="visual_mesh_scale" value="1.0 1.0 1.0" />
-  <xacro:property name="collision_mesh_scale" value="1.0 1.0 1.0" />
+  <xacro:property name="visual_mesh_scale" value="1.0 1.0 1.0"/>
+  <xacro:property name="collision_mesh_scale" value="1.0 1.0 1.0"/>
   <!-- Link & Joint -->
   <xacro:macro name="arm" params="prefix parent *joint_origin">
@@ -14,127 +14,125 @@
       <visual>
         <geometry>
-          <mesh filename="package://catchrobo_description/mesh/arm/link0.stl" scale="${visual_mesh_scale}" />
+          <mesh filename="package://catchrobo_description/mesh/arm/visual/link0.stl" scale="${visual_mesh_scale}"/>
         </geometry>
-        <material name="orange" />
+        <material name="white"/>
       </visual>
       <collision>
         <geometry>
-          <mesh filename="package://catchrobo_description/mesh/arm/link0.stl" scale="${collision_mesh_scale}" />
+          <mesh filename="package://catchrobo_description/mesh/arm/collision/link0.stl" scale="${collision_mesh_scale}"/>
         </geometry>
       </collision>
     </link>
     <joint name="${prefix}arm/joint1" type="revolute">
-      <parent link="${prefix}arm/link0" />
-      <child link="${prefix}arm/link1" />
-      <origin xyz="0 0 0.08" rpy="0 0 0" />
-      <axis xyz="0 0 1" />
-      <limit lower="${-150*M_PI/180}" upper="${150*M_PI/180}" effort="6" velocity="5" acceleration="5" />
+      <parent link="${prefix}arm/link0"/>
+      <child link="${prefix}arm/link1"/>
+      <origin xyz="0 0 0.1675" rpy="0 0 0"/>
+      <axis xyz="0 0 1"/>
+      <limit lower="${-160*M_PI/180}" upper="${160*M_PI/180}" effort="6"
+              velocity="5" acceleration="5"/>
     </joint>
     <link name="${prefix}arm/link1">
       <visual>
         <geometry>
-          <mesh filename="package://catchrobo_description/mesh/arm/link1.stl" scale="${visual_mesh_scale}" />
+          <mesh filename="package://catchrobo_description/mesh/arm/visual/link1.stl" scale="${visual_mesh_scale}"/>
         </geometry>
-        <material name="orange" />
+        <material name="white"/>
       </visual>
       <collision>
         <geometry>
-          <mesh filename="package://catchrobo_description/mesh/arm/link1.stl" scale="${collision_mesh_scale}" />
+          <mesh filename="package://catchrobo_description/mesh/arm/collision/link1.stl" scale="${collision_mesh_scale}"/>
         </geometry>
       </collision>
     </link>
     <joint name="${prefix}arm/joint2" type="revolute">
-      <parent link="${prefix}arm/link1" />
-      <child link="${prefix}arm/link2" />
-      <origin xyz="0 0 0.08" rpy="${90*M_PI/180} 0 ${90*M_PI/180}" />
-      <axis xyz="0 0 1" />
-      <limit lower="${-90*M_PI/180}" upper="${90*M_PI/180}" effort="6" velocity="5" acceleration="5" />
+      <parent link="${prefix}arm/link1"/>
+      <child link="${prefix}arm/link2"/>
+      <origin xyz="0 0 0" rpy="${90*M_PI/180} 0 0"/>
+      <axis xyz="0 0 1"/>
+      <limit lower="${-90*M_PI/180}" upper="${90*M_PI/180}" effort="6"
+              velocity="5" acceleration="5"/>
     </joint>
     <link name="${prefix}arm/link2">
       <visual>
         <geometry>
-          <mesh filename="package://catchrobo_description/mesh/arm/link2.stl" scale="${visual_mesh_scale}" />
+          <mesh filename="package://catchrobo_description/mesh/arm/visual/link2.stl" scale="${visual_mesh_scale}"/>
         </geometry>
-        <material name="orange" />
+        <material name="white"/>
       </visual>
       <collision>
         <geometry>
-          <mesh filename="package://catchrobo_description/mesh/arm/link2.stl" scale="${collision_mesh_scale}" />
+          <mesh filename="package://catchrobo_description/mesh/arm/collision/link2.stl" scale="${collision_mesh_scale}"/>
         </geometry>
       </collision>
     </link>
     <joint name="${prefix}arm/joint3" type="revolute">
-      <parent link="${prefix}arm/link2" />
-      <child link="${prefix}arm/link3" />
-      <origin xyz="0 0.45 0" rpy="0 0 0" />
-      <axis xyz="0 0 1" />
-      <limit lower="${-160*M_PI/180}" upper="0" effort="6" velocity="5" acceleration="5" />
+      <parent link="${prefix}arm/link2"/>
+      <child link="${prefix}arm/link3"/>
+      <origin xyz="0 0.44 0" rpy="0 0 0"/>
+      <axis xyz="0 0 1"/>
+      <limit lower="${-160*M_PI/180}" upper="${0*M_PI/180}" effort="6"
+              velocity="5" acceleration="5"/>
     </joint>
     <link name="${prefix}arm/link3">
       <visual>
         <geometry>
-          <mesh filename="package://catchrobo_description/mesh/arm/link3.stl" scale="${visual_mesh_scale}" />
+          <mesh filename="package://catchrobo_description/mesh/arm/visual/link3.stl" scale="${visual_mesh_scale}"/>
         </geometry>
-        <material name="orange" />
+        <material name="white"/>
       </visual>
       <collision>
         <geometry>
-          <mesh filename="package://catchrobo_description/mesh/arm/link3.stl" scale="${collision_mesh_scale}" />
+          <mesh filename="package://catchrobo_description/mesh/arm/collision/link3.stl" scale="${collision_mesh_scale}"/>
         </geometry>
       </collision>
     </link>
     <joint name="${prefix}arm/joint4" type="revolute">
-      <parent link="${prefix}arm/link3" />
-      <child link="${prefix}arm/link4" />
-      <origin xyz="0 0.45 0" rpy="0 0 0" />
-      <axis xyz="0 0 1" />
-      <limit lower="${-90*M_PI/180}" upper="${90*M_PI/180}" effort="6" velocity="5" acceleration="5" />
+      <parent link="${prefix}arm/link3"/>
+      <child link="${prefix}arm/link4"/>
+      <origin xyz="0 0.44 0" rpy="0 0 0"/>
+      <axis xyz="0 0 1"/>
+      <limit lower="${-90*M_PI/180}" upper="${90*M_PI/180}" effort="6"
+              velocity="5" acceleration="5"/>
     </joint>
     <link name="${prefix}arm/link4">
       <visual>
         <geometry>
-          <mesh filename="package://catchrobo_description/mesh/arm/link4.stl" scale="${visual_mesh_scale}" />
+          <mesh filename="package://catchrobo_description/mesh/arm/visual/link4.stl" scale="${visual_mesh_scale}"/>
         </geometry>
-        <material name="orange" />
+        <material name="white"/>
       </visual>
       <collision>
         <geometry>
-          <mesh filename="package://catchrobo_description/mesh/arm/link4.stl" scale="${collision_mesh_scale}" />
+          <mesh filename="package://catchrobo_description/mesh/arm/collision/link4.stl" scale="${collision_mesh_scale}"/>
         </geometry>
       </collision>
     </link>
     <joint name="${prefix}arm/joint5" type="revolute">
-      <parent link="${prefix}arm/link4" />
-      <child link="${prefix}arm/link5" />
-      <origin xyz="0 0.04 0" rpy="${-90*M_PI/180} 0 0" />
-      <axis xyz="0 0 1" />
-      <limit lower="${-150*M_PI/180}" upper="${150*M_PI/180}" effort="6" velocity="5" acceleration="5" />
+      <parent link="${prefix}arm/link4"/>
+      <child link="${prefix}arm/link5"/>
+      <origin xyz="0 0.046 0" rpy="${-90*M_PI/180} 0 0"/>
+      <axis xyz="0 0 1"/>
+      <limit lower="${-160*M_PI/180}" upper="${160*M_PI/180}" effort="6"
+              velocity="5" acceleration="5"/>
     </joint>
     <link name="${prefix}arm/link5">
       <visual>
         <geometry>
-          <mesh filename="package://catchrobo_description/mesh/arm/link5.stl" scale="${visual_mesh_scale}" />
+          <mesh filename="package://catchrobo_description/mesh/arm/visual/link5.stl" scale="${visual_mesh_scale}"/>
         </geometry>
-        <material name="orange" />
+        <material name="white"/>
       </visual>
       <collision>
         <geometry>
-          <mesh filename="package://catchrobo_description/mesh/arm/link5.stl" scale="${collision_mesh_scale}" />
+          <mesh filename="package://catchrobo_description/mesh/arm/collision/link5.stl" scale="${collision_mesh_scale}"/>
         </geometry>
       </collision>
     </link>
     <joint name="${prefix}arm/joint_tip" type="fixed">
-      <parent link="${prefix}arm/link5" />
-      <child link="${prefix}arm/link_tip" />
-      <origin xyz="0 0 0.02" rpy="0 0 0" />
+      <parent link="${prefix}arm/link5"/>
+      <child link="${prefix}arm/link_tip"/>
+      <origin xyz="0 0 0.001" rpy="0 0 0"/>
     </joint>
-    <link name="${prefix}arm/link_tip" />
-    <!-- Transmissions -->
-    <!-- <xacro:include filename="$(find catchrobo_description)/urdf/arm.transmission.xacro" />
-    <arm_simple_transmission id="1" reduction="1.0" />
-    <arm_simple_transmission id="2" reduction="1.0" />
-    <arm_simple_transmission id="3" reduction="1.0" />
-    <arm_simple_transmission id="4" reduction="1.0" />
-    <arm_simple_transmission id="5" reduction="1.0" /> -->
+    <link name="${prefix}arm/link_tip"/>
   </xacro:macro>
 </robot>

File: catchrobo_description/urdf/base.urdf.xacro (robot description, xacro)
@@ -2,27 +2,27 @@
 <robot xmlns:xacro="http://ros.org/wiki/xacro">
   <!-- Field Side Parameters-->
-  <xacro:arg name="field" default="" />
+  <xacro:arg name="field" default=""/>
   <xacro:property name="field" value="$(arg field)" />
   <!-- Constants -->
-  <xacro:property name="visual_mesh_scale" value="1.0 1.0 1.0" />
-  <xacro:property name="collision_mesh_scale" value="1.0 1.0 1.0" />
+  <xacro:property name="visual_mesh_scale" value="1.0 1.0 1.0"/>
+  <xacro:property name="collision_mesh_scale" value="1.0 1.0 1.0"/>
   <!-- Link & Joint -->
   <xacro:macro name="base" params="parent *joint_origin">
     <joint name="base/root" type="fixed">
-      <xacro:insert_block name="joint_origin" />
-      <parent link="${parent}" />
-      <child link="base/base_link" />
+      <xacro:insert_block name="joint_origin"/>
+      <parent link="${parent}"/>
+      <child link="base/base_link"/>
     </joint>
-    <!-- <link name="base/base_link">
+    <link name="base/base_link">
       <xacro:if value="${field=='blue'}">
         <visual>
           <geometry>
-            <mesh filename="package://catchrobo_description/mesh/base/base_blue.stl" scale="${visual_mesh_scale}" />
+            <mesh filename="package://catchrobo_description/mesh/base/visual/base_blue_plane.stl" scale="${visual_mesh_scale}"/>
           </geometry>
-          <material name="white" />
+          <material name="white"/>
         </visual>
         <collision>
           <geometry>
-            <mesh filename="package://catchrobo_description/mesh/base/base_blue.stl" scale="${collision_mesh_scale}" />
+            <mesh filename="package://catchrobo_description/mesh/base/collision/base_blue_plane.stl" scale="${collision_mesh_scale}"/>
           </geometry>
         </collision>
@@ -31,39 +31,11 @@
         <visual>
           <geometry>
-            <mesh filename="package://catchrobo_description/mesh/base/base_red.stl" scale="${visual_mesh_scale}" />
+            <mesh filename="package://catchrobo_description/mesh/base/visual/base_red_plane.stl" scale="${visual_mesh_scale}"/>
           </geometry>
-          <material name="white" />
+          <material name="white"/>
         </visual>
         <collision>
           <geometry>
-            <mesh filename="package://catchrobo_description/mesh/base/base_red.stl" scale="${collision_mesh_scale}" />
-          </geometry>
-        </collision>
-      </xacro:if>
-    </link> -->
-    <link name="base/base_link">
-      <xacro:if value="${field=='blue'}">
-        <visual>
-          <geometry>
-            <mesh filename="package://catchrobo_description/mesh/base/blue_side_without_bisco_re.stl.stl" scale="${visual_mesh_scale}" />
-          </geometry>
-          <material name="white" />
-        </visual>
-        <collision>
-          <geometry>
-            <mesh filename="package://catchrobo_description/mesh/base/blue_side_without_bisco_re.stl.stl" scale="${collision_mesh_scale}" />
-          </geometry>
-        </collision>
-      </xacro:if>
-      <xacro:if value="${field=='red'}">
-        <visual>
-          <geometry>
-            <mesh filename="package://catchrobo_description/mesh/base/red_side_without_bisco_re.stl" scale="${visual_mesh_scale}" />
-          </geometry>
-          <material name="white" />
-        </visual>
-        <collision>
-          <geometry>
-            <mesh filename="package://catchrobo_description/mesh/base/red_side_without_bisco_re.stl" scale="${collision_mesh_scale}" />
+            <mesh filename="package://catchrobo_description/mesh/base/collision/base_red_plane.stl" scale="${collision_mesh_scale}"/>
           </geometry>
         </collision>
@@ -71,14 +43,14 @@
     </link>
     <joint name="base/joint_tip" type="fixed">
-      <parent link="base/base_link" />
-      <child link="base/link_tip" />
+      <parent link="base/base_link"/>
+      <child link="base/link_tip"/>
       <xacro:if value="${field=='blue'}">
-        <origin xyz="-0.8 0.4 0.0044" rpy="0 0 0" />
+        <origin xyz="-0.795 0.390 0.0044" rpy="0 0 0"/>
       </xacro:if>
       <xacro:if value="${field=='red'}">
-        <origin xyz="0.8 0.4 0.0044" rpy="0 0 0" />
+        <origin xyz="0.795 0.390 0.0044" rpy="0 0 ${180*M_PI/180}"/>
       </xacro:if>
     </joint>
-    <link name="base/link_tip" />
+    <link name="base/link_tip"/>
   </xacro:macro>
 </robot>

File: catchrobo_description/urdf/gripper.urdf.xacro (robot description, xacro)
@@ -14,39 +14,40 @@
       <visual>
         <geometry>
-          <mesh filename="package://catchrobo_description/mesh/gripper/base_link.stl" scale="${visual_mesh_scale}"/>
+          <mesh filename="package://catchrobo_description/mesh/gripper/visual/base_link.stl" scale="${visual_mesh_scale}"/>
         </geometry>
-        <material name="green"/>
+        <material name="white"/>
       </visual>
       <collision>
         <geometry>
-          <mesh filename="package://catchrobo_description/mesh/gripper/base_link.stl" scale="${collision_mesh_scale}"/>
+          <mesh filename="package://catchrobo_description/mesh/gripper/collision/base_link.stl" scale="${collision_mesh_scale}"/>
         </geometry>
       </collision>
     </link>
+    <!-- Gripper 1 -->
     <joint name="${prefix}gripper/joint1" type="prismatic">
       <parent link="${prefix}gripper/base_link"/>
-      <child link="${prefix}gripper/finger1"/>
-      <origin xyz="0 -0.05 0.01" rpy="${90*M_PI/180} 0 ${180*M_PI/180}"/>
+      <child link="${prefix}gripper/finger1_1"/>
+      <origin xyz="0.06 -0.05 0.02335" rpy="${90*M_PI/180} 0 ${-90*M_PI/180}"/>
       <axis xyz="0 0 1"/>
       <limit lower="0" upper="0.05" effort="6"
               velocity="5" acceleration="5"/>
     </joint>
-    <link name="${prefix}gripper/finger1">
+    <link name="${prefix}gripper/finger1_1">
       <visual>
         <geometry>
-          <mesh filename="package://catchrobo_description/mesh/gripper/finger1.stl" scale="${visual_mesh_scale}"/>
+          <mesh filename="package://catchrobo_description/mesh/gripper/visual/finger.stl" scale="${visual_mesh_scale}"/>
         </geometry>
-        <material name="green"/>
+        <material name="orange"/>
       </visual>
       <collision>
         <geometry>
-          <mesh filename="package://catchrobo_description/mesh/gripper/finger1.stl" scale="${collision_mesh_scale}"/>
+          <mesh filename="package://catchrobo_description/mesh/gripper/collision/finger.stl" scale="${collision_mesh_scale}"/>
         </geometry>
       </collision>
     </link>
-    <joint name="${prefix}gripper/joint2" type="prismatic">
+    <joint name="${prefix}gripper/joint1_mimic" type="prismatic">
       <parent link="${prefix}gripper/base_link"/>
-      <child link="${prefix}gripper/finger2"/>
-      <origin xyz="0 0.05 0.01" rpy="${90*M_PI/180} 0 0"/>
+      <child link="${prefix}gripper/finger1_2"/>
+      <origin xyz="-0.06 -0.05 0.02335" rpy="${90*M_PI/180} 0 ${90*M_PI/180}"/>
       <axis xyz="0 0 1"/>
       <limit lower="0" upper="0.05" effort="6"
@@ -54,23 +55,73 @@
       <mimic joint="${prefix}gripper/joint1" multiplier="1" offset="0" />
     </joint>
-    <link name="${prefix}gripper/finger2">
+    <link name="${prefix}gripper/finger1_2">
       <visual>
         <geometry>
-          <mesh filename="package://catchrobo_description/mesh/gripper/finger2.stl" scale="${visual_mesh_scale}"/>
+          <mesh filename="package://catchrobo_description/mesh/gripper/visual/finger.stl" scale="${visual_mesh_scale}"/>
         </geometry>
-        <material name="green"/>
+        <material name="orange"/>
       </visual>
       <collision>
         <geometry>
-          <mesh filename="package://catchrobo_description/mesh/gripper/finger2.stl" scale="${collision_mesh_scale}"/>
+          <mesh filename="package://catchrobo_description/mesh/gripper/collision/finger.stl" scale="${collision_mesh_scale}"/>
         </geometry>
       </collision>
     </link>
-    <joint name="${prefix}gripper/joint_tip" type="fixed">
+    <joint name="${prefix}gripper/grasping_frame1_joint" type="fixed">
       <parent link="${prefix}gripper/base_link"/>
-      <child link="${prefix}gripper/link_tip"/>
-      <origin xyz="0 0 0.03" rpy="0 0 0"/>
+      <child link="${prefix}gripper/grasping_frame1"/>
+      <origin xyz="0 -0.05 0.04835" rpy="0 0 0"/>
     </joint>
-    <link name="${prefix}gripper/link_tip"/>
+    <link name="${prefix}gripper/grasping_frame1"/>
+    <!-- Gripper 2 -->
+    <joint name="${prefix}gripper/joint2" type="prismatic">
+      <parent link="${prefix}gripper/base_link"/>
+      <child link="${prefix}gripper/finger2_1"/>
+      <origin xyz="0.06 0.05 0.02335" rpy="${90*M_PI/180} 0 ${-90*M_PI/180}"/>
+      <axis xyz="0 0 1"/>
+      <limit lower="0" upper="0.05" effort="6"
+              velocity="5" acceleration="5"/>
+    </joint>
+    <link name="${prefix}gripper/finger2_1">
+      <visual>
+        <geometry>
+          <mesh filename="package://catchrobo_description/mesh/gripper/visual/finger.stl" scale="${visual_mesh_scale}"/>
+        </geometry>
+        <material name="orange"/>
+      </visual>
+      <collision>
+        <geometry>
+          <mesh filename="package://catchrobo_description/mesh/gripper/collision/finger.stl" scale="${collision_mesh_scale}"/>
+        </geometry>
+      </collision>
+    </link>
+    <joint name="${prefix}gripper/joint2_mimic" type="prismatic">
+      <parent link="${prefix}gripper/base_link"/>
+      <child link="${prefix}gripper/finger2_2"/>
+      <origin xyz="-0.06 0.05 0.02335" rpy="${90*M_PI/180} 0 ${90*M_PI/180}"/>
+      <axis xyz="0 0 1"/>
+      <limit lower="0" upper="0.05" effort="6"
+              velocity="5" acceleration="5"/>
+      <mimic joint="${prefix}gripper/joint2" multiplier="1" offset="0" />
+    </joint>
+    <link name="${prefix}gripper/finger2_2">
+      <visual>
+        <geometry>
+          <mesh filename="package://catchrobo_description/mesh/gripper/visual/finger.stl" scale="${visual_mesh_scale}"/>
+        </geometry>
+        <material name="orange"/>
+      </visual>
+      <collision>
+        <geometry>
+          <mesh filename="package://catchrobo_description/mesh/gripper/collision/finger.stl" scale="${collision_mesh_scale}"/>
+        </geometry>
+      </collision>
+    </link>
+    <joint name="${prefix}gripper/grasping_frame2_joint" type="fixed">
+      <parent link="${prefix}gripper/base_link"/>
+      <child link="${prefix}gripper/grasping_frame2"/>
+      <origin xyz="0 0.05 0.04835" rpy="0 0 0"/>
+    </joint>
+    <link name="${prefix}gripper/grasping_frame2"/>
   </xacro:macro>
 </robot>

Commit message: scara urdf

File: catchrobo_description/robots/catchrobo.urdf.xacro (robot description, xacro)
@@ -8,4 +8,5 @@
   <xacro:include filename="$(find catchrobo_description)/urdf/base.urdf.xacro" />
   <xacro:include filename="$(find catchrobo_description)/urdf/arm.urdf.xacro" />
+  <xacro:include filename="$(find catchrobo_description)/urdf/scara.urdf.xacro" />
   <xacro:include filename="$(find catchrobo_description)/urdf/gripper.urdf.xacro" />
   <!-- Link & Joint -->
@@ -14,7 +15,10 @@
     <origin xyz="0 0 0" rpy="0 0 0" />
   </xacro:base>
-  <xacro:arm prefix="" parent="base/link_tip">
+  <!--<xacro:arm prefix="" parent="base/link_tip">
     <origin xyz="0 0 0" rpy="0 0 0" />
-  </xacro:arm>
+  </xacro:arm>-->
+  <xacro:scara prefix="" parent="base/link_tip">
+    <origin xyz="0 0 0.23" rpy="0 0 0" />
+  </xacro:scara>
   <xacro:gripper prefix="" parent="arm/link_tip">
     <origin xyz="0 0 0" rpy="0 0 0" />

Commit message: [Minor] Add shooter in catchrobo urdf (feature_shooter_urdf)

File: catchrobo_description/robots/catchrobo.urdf.xacro (robot description, xacro)
@@ -10,4 +10,5 @@
   <xacro:include filename="$(find catchrobo_description)/urdf/scara.urdf.xacro" />
   <xacro:include filename="$(find catchrobo_description)/urdf/gripper.urdf.xacro" />
+  <xacro:include filename="$(find catchrobo_description)/urdf/shooter.urdf.xacro" />
   <!-- Link & Joint -->
   <link name="world" />
@@ -24,3 +25,6 @@
     <origin xyz="0 0 0" rpy="0 0 0" />
   </xacro:gripper>
+  <xacro:shooter_base prefix="" parent="base/link_frame">
+    <origin xyz="0 0 0" rpy="0 0 0" />
+  </xacro:shooter_base>
 </robot>

File: catchrobo_description/urdf/base.urdf.xacro (robot description, xacro)
@@ -53,4 +53,15 @@
     </joint>
     <link name="base/link_tip"/>
+    <joint name="base/joint_frame" type="fixed">
+      <parent link="base/base_link"/>
+      <child link="base/link_frame"/>
+      <xacro:if value="${field=='blue'}">
+        <origin xyz="-1.1775 0.295 -0.0116" rpy="0 0 0"/>
+      </xacro:if>
+      <xacro:if value="${field=='red'}">
+        <origin xyz="1.1775 0.295 -0.0116" rpy="0 0 0"/>
+      </xacro:if>
+    </joint>
+    <link name="base/link_frame"/>
   </xacro:macro>
 </robot>

File: catchrobo_description/urdf/shooter.urdf.xacro (robot description, xacro)
@@ -46,5 +46,4 @@
       <parent link="${prefix}shooter_base/base_link"/>
       <child link="${prefix}shooter/guide"/>
-      <!--<origin xyz="0.3083 0.42041555 0.07832442" rpy="0 ${90*M_PI/180} ${-125*M_PI/180}"/>-->
       <origin xyz="0.3083 0.42041555 0.07832442" rpy="${-90*M_PI/180} ${35*M_PI/180} ${90*M_PI/180}"/>
       <axis xyz="0 0 1"/>
