Commit message: scara moveit  setup

File: catchrobo_description/robots/catchrobo.urdf.xacro (robot description, xacro)
@@ -25,6 +25,6 @@
     <origin xyz="0 0 0" rpy="0 0 0" />
   </xacro:gripper>
-  <xacro:shooter_base prefix="" parent="base/link_frame">
+  <xacro:shooter prefix="" parent="base/link_frame">
     <origin xyz="0 0 0" rpy="0 0 0" />
-  </xacro:shooter_base>
+  </xacro:shooter>
 </robot>

File: catchrobo_description/urdf/shooter.urdf.xacro (robot description, xacro)
@@ -7,42 +7,26 @@
   <xacro:property name="visual_mesh_scale" value="1.0 1.0 1.0"/>
   <xacro:property name="collision_mesh_scale" value="1.0 1.0 1.0"/>
-  <xacro:include filename="$(find catchrobo_description)/urdf/shooter.transmission.xacro"/>
   <!-- Link & Joint -->
-  <xacro:macro name="shooter_base" params="prefix parent *joint_origin">
-    <joint name="${prefix}shooter_base/root" type="fixed">
+  <xacro:macro name="shooter" params="prefix parent *joint_origin">
+    <joint name="${prefix}shooter/root" type="fixed">
       <xacro:insert_block name="joint_origin"/>
       <parent link="${parent}"/>
-      <child link="${prefix}shooter_base/base_link"/>
+      <child link="${prefix}shooter/base_link"/>
     </joint>
-    <link name="${prefix}shooter_base/base_link">
-      <xacro:if value="${field=='blue'}">
-        <visual>
-          <geometry>
-            <mesh filename="package://catchrobo_description/mesh/shooter/visual/shooter_base_fixed_axis.stl" scale="${visual_mesh_scale}"/>
-          </geometry>
-          <material name="white"/>
-        </visual>
-        <collision>
-          <geometry>
-            <mesh filename="package://catchrobo_description/mesh/shooter/collision/shooter_base_fixed_axis.stl" scale="${collision_mesh_scale}"/>
-          </geometry>
-        </collision>
-      </xacro:if>
-      <xacro:if value="${field=='red'}">
-        <visual>
-          <geometry>
-            <mesh filename="package://catchrobo_description/mesh/shooter/visual/shooter_base_fixed_axis.stl" scale="${visual_mesh_scale}"/>
-          </geometry>
-          <material name="white"/>
-        </visual>
-        <collision>
-          <geometry>
-            <mesh filename="package://catchrobo_description/mesh/shooter/collision/shooter_base_fixed_axis.stl" scale="${collision_mesh_scale}"/>
-          </geometry>
-        </collision>
-      </xacro:if>
+    <link name="${prefix}shooter/base_link">
+      <visual>
+        <geometry>
+          <mesh filename="package://catchrobo_description/mesh/shooter/visual/base.stl" scale="${visual_mesh_scale}"/>
+        </geometry>
+        <material name="white"/>
+      </visual>
+      <collision>
+        <geometry>
+          <mesh filename="package://catchrobo_description/mesh/shooter/collision/base.stl" scale="${collision_mesh_scale}"/>
+        </geometry>
+      </collision>
     </link>
-    <joint name="${prefix}shooter/joint1" type="revolute">
-      <parent link="${prefix}shooter_base/base_link"/>
+    <joint name="${prefix}guide/joint1" type="revolute">
+      <parent link="${prefix}shooter/base_link"/>
       <child link="${prefix}shooter/guide"/>
       <origin xyz="0.3083 0.42041555 0.07832442" rpy="${-90*M_PI/180} ${35*M_PI/180} ${90*M_PI/180}"/>
@@ -64,6 +48,6 @@
       </collision>
     </link>
-    <joint name="${prefix}shooter/joint2" type="revolute">
-      <parent link="${prefix}shooter_base/base_link"/>
+    <joint name="${prefix}sorter/joint1" type="revolute">
+      <parent link="${prefix}shooter/base_link"/>
       <child link="${prefix}shooter/sorter1"/>
       <origin xyz="0.195 0.41552443 0.01729232" rpy="0 ${35*M_PI/180} ${90*M_PI/180}"/>
@@ -85,6 +69,6 @@
       </collision>
     </link>
-    <joint name="${prefix}shooter/joint3" type="revolute">
-      <parent link="${prefix}shooter_base/base_link"/>
+    <joint name="${prefix}sorter/joint2" type="revolute">
+      <parent link="${prefix}shooter/base_link"/>
       <child link="${prefix}shooter/sorter2"/>
       <origin xyz="0 0.41552443 0.01729232" rpy="0 ${35*M_PI/180} ${90*M_PI/180}"/>
@@ -106,6 +90,6 @@
       </collision>
     </link>
-    <joint name="${prefix}shooter/joint4" type="revolute">
-      <parent link="${prefix}shooter_base/base_link"/>
+    <joint name="${prefix}sorter/joint3" type="revolute">
+      <parent link="${prefix}shooter/base_link"/>
       <child link="${prefix}shooter/sorter3"/>
       <origin xyz="-0.195 0.41552443 0.01729232" rpy="0 ${35*M_PI/180} ${90*M_PI/180}"/>

Commit message: scara  urdf update

File: catchrobo_description/robots/catchrobo.urdf.xacro (robot description, xacro)
@@ -19,11 +19,11 @@
     <origin xyz="0 0 0" rpy="0 0 0" />
   </xacro:arm>-->
-  <xacro:scara prefix="" parent="base/link_tip">
-    <origin xyz="0 0 0.23" rpy="0 0 0" />
+  <xacro:scara prefix="" parent="base/robot_tip">
+    <origin xyz="0 0 0" rpy="0 0 0" />
   </xacro:scara>
   <xacro:gripper prefix="" parent="arm/link_tip">
     <origin xyz="0 0 0" rpy="0 0 0" />
   </xacro:gripper>
-  <xacro:shooter prefix="" parent="base/link_frame">
+  <xacro:shooter prefix="" parent="base/shooter_tip">
     <origin xyz="0 0 0" rpy="0 0 0" />
   </xacro:shooter>

File: catchrobo_description/urdf/base.urdf.xacro (robot description, xacro)
@@ -42,7 +42,7 @@
       </xacro:if>
     </link>
-    <joint name="base/joint_tip" type="fixed">
+    <joint name="base/robot_tip" type="fixed">
       <parent link="base/base_link"/>
-      <child link="base/link_tip"/>
+      <child link="base/robot_tip"/>
       <xacro:if value="${field=='blue'}">
         <origin xyz="-0.795 0.390 0.0044" rpy="0 0 0"/>
@@ -52,8 +52,8 @@
       </xacro:if>
     </joint>
-    <link name="base/link_tip"/>
-    <joint name="base/joint_frame" type="fixed">
+    <link name="base/robot_tip"/>
+    <joint name="base/shooter_tip" type="fixed">
       <parent link="base/base_link"/>
-      <child link="base/link_frame"/>
+      <child link="base/shooter_tip"/>
       <xacro:if value="${field=='blue'}">
         <origin xyz="-1.1775 0.295 -0.0116" rpy="0 0 0"/>
@@ -63,5 +63,43 @@
       </xacro:if>
     </joint>
-    <link name="base/link_frame"/>
+    <link name="base/shooter_tip"/>
+    <joint name="base/pc" type="fixed">
+      <parent link="base/base_link"/>
+      <child link="base/pc"/>
+      <xacro:if value="${field=='blue'}">
+        <origin xyz="-0.85 0 0.2" rpy="0 0 0"/>
+      </xacro:if>
+      <xacro:if value="${field=='red'}">
+        <origin xyz="0.85 0 0.2" rpy="0 0 0"/>
+      </xacro:if>
+    </joint>
+    <link name="base/pc">
+      <visual>
+        <geometry>
+          <box size="0.25 0.4 0.4"/>
+        </geometry>
+        <origin xyz="0 0 0" rpy="0 0 0"/>
+        <material name="grey"/>
+      </visual>
+    </link>
+    <joint name="base/entry_prohibited_area" type="fixed">
+      <parent link="base/base_link"/>
+      <child link="base/entry_prohibited_area"/>
+      <xacro:if value="${field=='blue'}">
+        <origin xyz="0.2 0.7 0.4" rpy="0 0 0"/>
+      </xacro:if>
+      <xacro:if value="${field=='red'}">
+        <origin xyz="-0.2 0.7 0.4" rpy="0 0 0"/>
+      </xacro:if>
+    </joint>
+    <link name="base/entry_prohibited_area">
+      <visual>
+        <geometry>
+          <box size="0.1 2.0 0.8"/>
+        </geometry>
+        <origin xyz="0 0 0" rpy="0 0 0"/>
+        <material name="entry_prohibited_area"/>
+      </visual>
+    </link>
   </xacro:macro>
 </robot>

File: catchrobo_description/urdf/gripper.urdf.xacro (robot description, xacro)
@@ -14,5 +14,5 @@
       <visual>
         <geometry>
-          <mesh filename="package://catchrobo_description/mesh/gripper/visual/base_link.stl" scale="${visual_mesh_scale}"/>
+          <mesh filename="package://catchrobo_description/mesh/gripper/visual/base.stl" scale="${visual_mesh_scale}"/>
         </geometry>
         <material name="white"/>
@@ -20,5 +20,5 @@
       <collision>
         <geometry>
-          <mesh filename="package://catchrobo_description/mesh/gripper/collision/base_link.stl" scale="${collision_mesh_scale}"/>
+          <mesh filename="package://catchrobo_description/mesh/gripper/collision/base.stl" scale="${collision_mesh_scale}"/>
         </geometry>
       </collision>
@@ -28,5 +28,5 @@
       <parent link="${prefix}gripper/base_link"/>
       <child link="${prefix}gripper/finger1_1"/>
-      <origin xyz="0.06 -0.05 0.02335" rpy="${90*M_PI/180} 0 ${-90*M_PI/180}"/>
+      <origin xyz="0.06 -0.05 0.02035" rpy="${90*M_PI/180} 0 ${-90*M_PI/180}"/>
       <axis xyz="0 0 1"/>
       <limit lower="0" upper="0.05" effort="6"
@@ -49,5 +49,5 @@
       <parent link="${prefix}gripper/base_link"/>
       <child link="${prefix}gripper/finger1_2"/>
-      <origin xyz="-0.06 -0.05 0.02335" rpy="${90*M_PI/180} 0 ${90*M_PI/180}"/>
+      <origin xyz="-0.06 -0.05 0.02035" rpy="${90*M_PI/180} 0 ${90*M_PI/180}"/>
       <axis xyz="0 0 1"/>
       <limit lower="0" upper="0.05" effort="6"
@@ -78,5 +78,5 @@
       <parent link="${prefix}gripper/base_link"/>
       <child link="${prefix}gripper/finger2_1"/>
-      <origin xyz="0.06 0.05 0.02335" rpy="${90*M_PI/180} 0 ${-90*M_PI/180}"/>
+      <origin xyz="0.06 0.05 0.02035" rpy="${90*M_PI/180} 0 ${-90*M_PI/180}"/>
       <axis xyz="0 0 1"/>
       <limit lower="0" upper="0.05" effort="6"
@@ -99,5 +99,5 @@
       <parent link="${prefix}gripper/base_link"/>
       <child link="${prefix}gripper/finger2_2"/>
-      <origin xyz="-0.06 0.05 0.02335" rpy="${90*M_PI/180} 0 ${90*M_PI/180}"/>
+      <origin xyz="-0.06 0.05 0.02035" rpy="${90*M_PI/180} 0 ${90*M_PI/180}"/>
       <axis xyz="0 0 1"/>
       <limit lower="0" upper="0.05" effort="6"

File: catchrobo_description/urdf/scara.urdf.xacro (robot description, xacro)
@@ -28,5 +28,5 @@
       <parent link="${prefix}arm/link0"/>
       <child link="${prefix}arm/link1"/>
-      <origin xyz="0 0 0.1062" rpy="0 0 0"/>
+      <origin xyz="0 0 0.3175" rpy="0 0 0"/>
       <axis xyz="0 0 1"/>
       <limit lower="${-160*M_PI/180}" upper="${160*M_PI/180}" effort="6"
@@ -49,5 +49,5 @@
       <parent link="${prefix}arm/link1"/>
       <child link="${prefix}arm/link2"/>
-      <origin xyz="0.45 0 0.026" rpy="0 0 0"/>
+      <origin xyz="0.45 0 0.043" rpy="0 0 0"/>
       <axis xyz="0 0 1"/>
       <limit lower="${-160*M_PI/180}" upper="${160*M_PI/180}" effort="6"
@@ -91,5 +91,5 @@
       <parent link="${prefix}arm/link3"/>
       <child link="${prefix}arm/link4"/>
-      <origin xyz="0 0 -0.0403" rpy="0 0 0"/>
+      <origin xyz="0 0 -0.0335" rpy="0 0 0"/>
       <axis xyz="0 0 1"/>
       <limit lower="-0.25" upper="0" effort="6"

File: catchrobo_description/urdf/shooter.urdf.xacro (robot description, xacro)
@@ -32,5 +32,5 @@
       <origin xyz="0.3083 0.4215627 0.07996272" rpy="${-90*M_PI/180} ${35*M_PI/180} ${90*M_PI/180}"/>
       <axis xyz="0 0 1"/>
-      <limit lower="${-175*M_PI/180}" upper="${175*M_PI/180}" effort="6"
+      <limit lower="${-180*M_PI/180}" upper="${0*M_PI/180}" effort="6"
               velocity="5" acceleration="5"/>
     </joint>
@@ -40,5 +40,5 @@
           <mesh filename="package://catchrobo_description/mesh/shooter/visual/guide.stl" scale="${visual_mesh_scale}"/>
         </geometry>
-        <material name="white"/>
+        <material name="orange"/>
       </visual>
       <collision>
@@ -53,5 +53,5 @@
       <origin xyz="0.195 0.41552443 0.01729232" rpy="0 ${35*M_PI/180} ${90*M_PI/180}"/>
       <axis xyz="0 0 1"/>
-      <limit lower="${-175*M_PI/180}" upper="${175*M_PI/180}" effort="6"
+      <limit lower="${-45*M_PI/180}" upper="${45*M_PI/180}" effort="6"
               velocity="5" acceleration="5"/>
     </joint>
@@ -61,5 +61,5 @@
           <mesh filename="package://catchrobo_description/mesh/shooter/visual/sorter.stl" scale="${visual_mesh_scale}"/>
         </geometry>
-        <material name="white"/>
+        <material name="orange"/>
       </visual>
       <collision>
@@ -74,5 +74,5 @@
       <origin xyz="0 0.41552443 0.01729232" rpy="0 ${35*M_PI/180} ${90*M_PI/180}"/>
       <axis xyz="0 0 1"/>
-      <limit lower="${-175*M_PI/180}" upper="${175*M_PI/180}" effort="6"
+      <limit lower="${-45*M_PI/180}" upper="${45*M_PI/180}" effort="6"
               velocity="5" acceleration="5"/>
     </joint>
@@ -82,5 +82,5 @@
           <mesh filename="package://catchrobo_description/mesh/shooter/visual/sorter.stl" scale="${visual_mesh_scale}"/>
         </geometry>
-        <material name="white"/>
+        <material name="orange"/>
       </visual>
       <collision>
@@ -95,5 +95,5 @@
       <origin xyz="-0.195 0.41552443 0.01729232" rpy="0 ${35*M_PI/180} ${90*M_PI/180}"/>
       <axis xyz="0 0 1"/>
-      <limit lower="${-175*M_PI/180}" upper="${175*M_PI/180}" effort="6"
+      <limit lower="${-45*M_PI/180}" upper="${45*M_PI/180}" effort="6"
               velocity="5" acceleration="5"/>
     </joint>
@@ -103,5 +103,5 @@
           <mesh filename="package://catchrobo_description/mesh/shooter/visual/sorter.stl" scale="${visual_mesh_scale}"/>
         </geometry>
-        <material name="white"/>
+        <material name="orange"/>
       </visual>
       <collision>

Commit message: shooter down for moving

File: catchrobo_description/robots/catchrobo.urdf.xacro (robot description, xacro)
@@ -26,5 +26,5 @@
   </xacro:gripper>
   <xacro:shooter prefix="" parent="base/shooter_tip">
-    <origin xyz="0 0 0" rpy="0 0 0" />
+    <origin xyz="0 0 -0.030" rpy="0 0 0" />
   </xacro:shooter>
 </robot>

File: catchrobo_description/urdf/base.urdf.xacro (robot description, xacro)
@@ -68,8 +68,8 @@
       <child link="base/pc"/>
       <xacro:if value="${field=='blue'}">
-        <origin xyz="-0.85 0 0.2" rpy="0 0 0"/>
+        <origin xyz="-0.85 0 0.12" rpy="0 0 0"/>
       </xacro:if>
       <xacro:if value="${field=='red'}">
-        <origin xyz="0.85 0 0.2" rpy="0 0 0"/>
+        <origin xyz="0.85 0 0.12" rpy="0 0 0"/>
       </xacro:if>
     </joint>
@@ -77,5 +77,5 @@
       <visual>
         <geometry>
-          <box size="0.25 0.4 0.4"/>
+          <box size="0.25 0.4 0.24"/>
         </geometry>
         <origin xyz="0 0 0" rpy="0 0 0"/>

File: catchrobo_description/urdf/scara.urdf.xacro (robot description, xacro)
@@ -51,6 +51,12 @@
       <origin xyz="0.45 0 0.043" rpy="0 0 0"/>
       <axis xyz="0 0 1"/>
-      <limit lower="${-160*M_PI/180}" upper="${160*M_PI/180}" effort="6"
+      <xacro:if value="${field=='blue'}">
+        <limit lower="${-90*M_PI/180}" upper="${160*M_PI/180}" effort="6"
               velocity="5" acceleration="5"/>
+      </xacro:if>
+      <xacro:if value="${field=='red'}">
+        <limit lower="${-160*M_PI/180}" upper="${90*M_PI/180}" effort="6"
+              velocity="5" acceleration="5"/>
+      </xacro:if>
     </joint>
     <link name="${prefix}arm/link2">

Commit message: mesh models decimated

File: catchrobo_description/robots/catchrobo.urdf.xacro (robot description, xacro)
@@ -26,5 +26,5 @@
   </xacro:gripper>
   <xacro:shooter prefix="" parent="base/shooter_tip">
-    <origin xyz="0 0 -0.030" rpy="0 0 0" />
+    <origin xyz="0 0 0" rpy="0 0 0" />
   </xacro:shooter>
 </robot>

File: catchrobo_description/urdf/scara.urdf.xacro (robot description, xacro)
@@ -28,5 +28,5 @@
       <parent link="${prefix}arm/link0"/>
       <child link="${prefix}arm/link1"/>
-      <origin xyz="0 0 0.3175" rpy="0 0 0"/>
+      <origin xyz="0 0 0.4325" rpy="0 0 0"/>
       <axis xyz="0 0 1"/>
       <limit lower="${-160*M_PI/180}" upper="${160*M_PI/180}" effort="6"
@@ -49,5 +49,5 @@
       <parent link="${prefix}arm/link1"/>
       <child link="${prefix}arm/link2"/>
-      <origin xyz="0.45 0 0.043" rpy="0 0 0"/>
+      <origin xyz="0.45 0 0.04308" rpy="0 0 0"/>
       <axis xyz="0 0 1"/>
       <xacro:if value="${field=='blue'}">
@@ -97,7 +97,7 @@
       <parent link="${prefix}arm/link3"/>
       <child link="${prefix}arm/link4"/>
-      <origin xyz="0 0 -0.0335" rpy="0 0 0"/>
+      <origin xyz="0 0 -0.03295" rpy="0 0 0"/>
       <axis xyz="0 0 1"/>
-      <limit lower="-0.25" upper="0" effort="6"
+      <limit lower="-0.35" upper="0" effort="6"
               velocity="5" acceleration="5"/>
     </joint>

Commit message: kyounokamichousei

File: catchrobo_description/robots/catchrobo.urdf.xacro (robot description, xacro)
@@ -20,5 +20,5 @@
   </xacro:arm>-->
   <xacro:scara prefix="" parent="base/robot_tip">
-    <origin xyz="0 0 0" rpy="0 0 0" />
+    <origin xyz="0 0 -0.02" rpy="0 0 0" />
   </xacro:scara>
   <xacro:gripper prefix="" parent="arm/link_tip">

Commit message: error odrive

File: catchrobo_description/robots/catchrobo.urdf.xacro (robot description, xacro)
@@ -20,5 +20,6 @@
   </xacro:arm>-->
   <xacro:scara prefix="" parent="base/robot_tip">
-    <origin xyz="0 0 -0.02" rpy="0 0 0" />
+    <!--<origin xyz="0 0 -0.02" rpy="0 0 0" />-->
+    <origin xyz="0 0 0.019" rpy="0 0 0" />
   </xacro:scara>
   <xacro:gripper prefix="" parent="arm/link_tip">
@@ -26,5 +27,6 @@
   </xacro:gripper>
   <xacro:shooter prefix="" parent="base/shooter_tip">
-    <origin xyz="0 0 0" rpy="0 0 0" />
+    <!--<origin xyz="0 0 0.0" rpy="0 0 0" />-->
+    <origin xyz="0 0 0.039" rpy="0 0 0" />
   </xacro:shooter>
 </robot>

Commit message: urdf not work

File: catchrobo_description/robots/catchrobo.urdf.xacro (robot description, xacro)
@@ -3,4 +3,6 @@
   <xacro:arg name="field" default="" />
   <xacro:property name="field" value="$(arg field)" />
+  <xacro:arg name="dummy" default="false" />
+  <xacro:property name="dummy" value="$(arg dummy)" />
   <!-- Dependencies -->
   <xacro:include filename="$(find catchrobo_description)/urdf/materials.xacro" />
@@ -20,6 +22,11 @@
   </xacro:arm>-->
   <xacro:scara prefix="" parent="base/robot_tip">
-    <!--<origin xyz="0 0 -0.02" rpy="0 0 0" />-->
-    <origin xyz="0 0 0.019" rpy="0 0 0" />
+      <!-- <xacro:if value="${dummy=='true'}">
+      <origin xyz="0 0 0.019" rpy="0 0 0" />
+    </xacro:if>
+    <xacro:if value="${dummy=='false'}">
+      <origin xyz="0 0 -0.02" rpy="0 0 0" />
+    </xacro:if> -->
+<origin xyz="0 0 0.019" rpy="0 0 0" />
   </xacro:scara>
   <xacro:gripper prefix="" parent="arm/link_tip">
@@ -27,6 +34,11 @@
   </xacro:gripper>
   <xacro:shooter prefix="" parent="base/shooter_tip">
-    <!--<origin xyz="0 0 0.0" rpy="0 0 0" />-->
-    <origin xyz="0 0 0.039" rpy="0 0 0" />
+    <!-- <xacro:if value="${dummy=='true'}">
+      <origin xyz="0 0 0.0" rpy="0 0 0" />
+    </xacro:if>
+    <xacro:if value="${dummy=='false'}">
+      <origin xyz="0 0 0.039" rpy="0 0 0" />
+    </xacro:if> -->
+    <origin xyz="0 0 0.0" rpy="0 0 0" />
   </xacro:shooter>
 </robot>

File: catchrobo_description/urdf/base.urdf.xacro (robot description, xacro)
@@ -4,4 +4,6 @@
   <xacro:arg name="field" default=""/>
   <xacro:property name="field" value="$(arg field)" />
+   <xacro:arg name="dummy" default="false" />
+  <xacro:property name="dummy" value="$(arg dummy)" />
   <!-- Constants -->
   <xacro:property name="visual_mesh_scale" value="1.0 1.0 1.0"/>
@@ -47,4 +49,10 @@
       <xacro:if value="${field=='blue'}">
         <origin xyz="-0.795 0.350 0.0044" rpy="0 0 0"/>
+        <!-- <xacro:if value="${dummy=='true'}">
+          <origin xyz="-0.795 0.350 0.0234" rpy="0 0 0"/>
+        </xacro:if>
+        <xacro:if value="${dummy=='false'}">
+          <origin xyz="-0.795 0.350 -0.0156" rpy="0 0 0"/>
+        </xacro:if> -->
       </xacro:if>
       <xacro:if value="${field=='red'}">

Commit message: testrun 2

File: catchrobo_description/robots/catchrobo.urdf.xacro (robot description, xacro)
@@ -28,5 +28,6 @@
       <origin xyz="0 0 -0.02" rpy="0 0 0" />
     </xacro:if> -->
-<origin xyz="0 0 0.019" rpy="0 0 0" />
+<!-- <origin xyz="0 0 0.019" rpy="0 0 0" /> -->
+<origin xyz="0 0 -0.02" rpy="0 0 0" />
   </xacro:scara>
   <xacro:gripper prefix="" parent="arm/link_tip">
@@ -35,10 +36,13 @@
   <xacro:shooter prefix="" parent="base/shooter_tip">
     <!-- <xacro:if value="${dummy=='true'}">
-      <origin xyz="0 0 0.0" rpy="0 0 0" />
+      <origin xyz="0 0 0.039" rpy="0 0 0" />
     </xacro:if>
     <xacro:if value="${dummy=='false'}">
-      <origin xyz="0 0 0.039" rpy="0 0 0" />
+      <origin xyz="0 0 0.0" rpy="0 0 0" />
     </xacro:if> -->
+    <!-- honnbann -->
     <origin xyz="0 0 0.0" rpy="0 0 0" />
+    <!-- ie -->
+          <!-- <origin xyz="0 0 0.039" rpy="0 0 0" /> -->
   </xacro:shooter>
 </robot>

Commit message: after test run 5

File: catchrobo_description/robots/catchrobo.urdf.xacro (robot description, xacro)
@@ -42,5 +42,5 @@
     </xacro:if> -->
     <!-- honnbann -->
-    <origin xyz="0 0 0.0" rpy="0 0 0" />
+    <origin xyz="0 0 0.016" rpy="0 0 0" />
     <!-- ie -->
           <!-- <origin xyz="0 0 0.039" rpy="0 0 0" /> -->
